File: psc_carrier_brd.kicad_pcb (KiCad board)
At the start: 2 copper layers, 241.3 x 171.4 mm, 20 parts, among them J1 1731130154, J2 0836149012, J3 6469028-1, J4 6469028-1, J5 39301022, J6 6469028-1, J7 0836149012, J8 0836149012, J9 0836149012

Commit message: finish up regulator section
Parts:
- removed D1: LED, LED_SMD:LED_0603_1608Metric
- removed the J1 at (258.3, 71.1)
- removed the J2 at (69.8, 66.5)
- removed J9: 0836149012, myparts:0836149012
- added C10: 0.1uF, Capacitor_SMD:C_0402_1005Metric, F.Cu at (281.1, 161.5)
- added C11: 10uF, Capacitor_SMD:C_0603_1608Metric, F.Cu at (277.1, 139.3)
- added C12: 0.1uF, Capacitor_SMD:C_0402_1005Metric, B.Cu at (261.6, 131.5)
- added C13: 0.1uF, Capacitor_SMD:C_0402_1005Metric, B.Cu at (264.2, 158.5)
- added C14: 0.1uF, Capacitor_SMD:C_0402_1005Metric, B.Cu at (261.7, 152.5)
- added C15: 0.1uF, Capacitor_SMD:C_0402_1005Metric, F.Cu at (279.1, 139.1)
- added C16: 100uF, myparts:CAP_EEFK_D8_PAN, F.Cu at (271.1, 174.5)
- added C17: 100uF, myparts:CAP_EEFK_D8_PAN, F.Cu at (271.4, 196.0)
- added C18: 10uF, Capacitor_SMD:C_0603_1608Metric, F.Cu at (279.5, 174.3)
- added C19: 10uF, Capacitor_SMD:C_0603_1608Metric, F.Cu at (279.7, 194.0)
- added C2: 100uF, myparts:CAP_EEFK_D8_PAN, F.Cu at (271.1, 147.5)
- added C20: 0.1uF, Capacitor_SMD:C_0402_1005Metric, F.Cu at (281.5, 174.7)
- added C21: 0.1uF, Capacitor_SMD:C_0402_1005Metric, F.Cu at (281.5, 194.6)
- added C22: 100uF, myparts:CAPMP7.6X4.3_4.3N_KEM, F.Cu at (270.8, 210.5)
- added C23: 100uF, myparts:CAPMP7.6X4.3_4.3N_KEM, F.Cu at (271.0, 189.0)
- added C24: 10uF, Capacitor_SMD:C_0603_1608Metric, F.Cu at (279.5, 210.3)
- added C25: 0.1uF, Capacitor_SMD:C_0402_1005Metric, F.Cu at (281.5, 210.0)
- added C26: 10uF, Capacitor_SMD:C_0603_1608Metric, F.Cu at (277.5, 187.8)
- added C27: 0.1uF, Capacitor_SMD:C_0402_1005Metric, F.Cu at (279.5, 187.6)
- added C28: 0.1uF, Capacitor_SMD:C_0402_1005Metric, B.Cu at (264.5, 207.0)
- added C29: 0.1uF, Capacitor_SMD:C_0402_1005Metric, B.Cu at (262.0, 201.0)
- added C3: 10uF, Capacitor_SMD:C_0603_1608Metric, F.Cu at (279.1, 125.8)
- added C30: 0.1uF, Capacitor_SMD:C_0402_1005Metric, B.Cu at (262.0, 180.0)
- added C31: 10uF, Capacitor_SMD:C_0603_1608Metric, F.Cu at (291.8, 265.0)
- added C32: 10uF, Capacitor_SMD:C_0603_1608Metric, F.Cu at (287.3, 265.0)
- added C33: 0.1uF, Capacitor_SMD:C_0402_1005Metric, F.Cu at (285.8, 264.7)
- added C34: 0.1uF, Capacitor_SMD:C_0402_1005Metric, F.Cu at (279.2, 265.2)
- added C35: 10uF, Capacitor_SMD:C_0603_1608Metric, F.Cu at (277.7, 265.4)
- added C36: 100uF, Capacitor_SMD:C_1206_3216Metric, F.Cu at (275.7, 266.2)
- added C37: 10uF, Capacitor_SMD:C_0603_1608Metric, F.Cu at (293.2, 292.0)
- added C38: 10uF, Capacitor_SMD:C_0603_1608Metric, F.Cu at (288.4, 292.0)
- added C39: 0.1uF, Capacitor_SMD:C_0402_1005Metric, F.Cu at (286.7, 291.8)
- added C4: 10uF, Capacitor_SMD:C_0603_1608Metric, F.Cu at (279.4, 145.5)
- added C40: 0.1uF, Capacitor_SMD:C_0402_1005Metric, F.Cu at (280.2, 293.8)
- added C41: 10uF, Capacitor_SMD:C_0603_1608Metric, F.Cu at (278.7, 294.1)
- added C42: 100uF, Capacitor_SMD:C_1206_3216Metric, F.Cu at (276.7, 294.8)
- added C43: 10uF, Capacitor_SMD:C_0603_1608Metric, F.Cu at (292.7, 315.9)
- added C44: 10uF, Capacitor_SMD:C_0603_1608Metric, F.Cu at (287.9, 315.9)
- added C45: 0.1uF, Capacitor_SMD:C_0402_1005Metric, F.Cu at (286.2, 315.7)
- added C46: 0.1uF, Capacitor_SMD:C_0402_1005Metric, F.Cu at (279.7, 317.7)
- added C47: 10uF, Capacitor_SMD:C_0603_1608Metric, F.Cu at (278.2, 318.0)
- added C48: 100uF, Capacitor_SMD:C_1206_3216Metric, F.Cu at (276.2, 318.7)
- added C49: 10uF, Capacitor_SMD:C_0603_1608Metric, F.Cu at (292.8, 303.9)
- added C5: 0.1uF, Capacitor_SMD:C_0402_1005Metric, F.Cu at (295.7, 127.4)
- added C50: 10uF, Capacitor_SMD:C_0603_1608Metric, F.Cu at (288.0, 303.9)
- added C51: 0.1uF, Capacitor_SMD:C_0402_1005Metric, F.Cu at (286.3, 303.7)
- added C52: 0.1uF, Capacitor_SMD:C_0402_1005Metric, F.Cu at (279.8, 305.7)
- added C53: 10uF, Capacitor_SMD:C_0603_1608Metric, F.Cu at (278.3, 306.0)
- added C54: 100uF, Capacitor_SMD:C_1206_3216Metric, F.Cu at (276.3, 306.7)
- added C55: 10uF, Capacitor_SMD:C_0603_1608Metric, F.Cu at (293.2, 280.4)
- added C56: 10uF, Capacitor_SMD:C_0603_1608Metric, F.Cu at (288.4, 280.4)
- added C57: 0.1uF, Capacitor_SMD:C_0402_1005Metric, F.Cu at (286.7, 280.2)
- added C58: 0.1uF, Capacitor_SMD:C_0402_1005Metric, F.Cu at (280.2, 282.2)
- added C59: 10uF, Capacitor_SMD:C_0603_1608Metric, F.Cu at (278.7, 282.5)
- added C6: 0.1uF, Capacitor_SMD:C_0402_1005Metric, F.Cu at (281.1, 146.1)
- added C60: 100uF, Capacitor_SMD:C_1206_3216Metric, F.Cu at (276.7, 283.2)
- added C61: 0.1uF, Capacitor_SMD:C_0402_1005Metric, B.Cu at (264.2, 227.3)
- added C62: 0.1uF, Capacitor_SMD:C_0402_1005Metric, B.Cu at (263.6, 274.3)
- added C63: 10uF, Capacitor_SMD:C_0603_1608Metric, F.Cu at (287.2, 252.7)
- added C64: 0.1uF, Capacitor_SMD:C_0402_1005Metric, F.Cu at (285.7, 252.5)
- added C65: 10uF, Capacitor_SMD:C_0603_1608Metric, F.Cu at (291.7, 252.7)
- added C66: 10uF, Capacitor_SMD:C_0603_1608Metric, F.Cu at (278.2, 253.2)
- added C67: 0.1uF, Capacitor_SMD:C_0402_1005Metric, F.Cu at (279.7, 252.9)
- added C68: 100uF, Capacitor_SMD:C_1206_3216Metric, F.Cu at (276.2, 253.7)
- added C69: 0.1uF, Capacitor_SMD:C_0402_1005Metric, F.Cu at (263.8, 227.3)
- added C7: 100uF, myparts:CAPMP7.6X4.3_4.3N_KEM, F.Cu at (270.5, 162.0)
- added C8: 100uF, myparts:CAPMP7.6X4.3_4.3N_KEM, F.Cu at (270.6, 140.5)
- added C9: 10uF, Capacitor_SMD:C_0603_1608Metric, F.Cu at (279.1, 161.8)
- added J6: 61083-061402LF, myparts:AMPHENOL_61083-061402LF, F.Cu at (95.0, 153.0)
- added L1: LSMGG160808T331RG, myparts:IND_LSMG_160808_TAY, F.Cu at (289.6, 264.2)
- added L2: LSMGG160808T331RG, myparts:IND_LSMG_160808_TAY, F.Cu at (291.0, 291.3)
- added L3: LSMGG160808T331RG, myparts:IND_LSMG_160808_TAY, F.Cu at (290.5, 315.2)
- added L4: LSMGG160808T331RG, myparts:IND_LSMG_160808_TAY, F.Cu at (290.6, 303.2)
- added L5: LSMGG160808T331RG, myparts:IND_LSMG_160808_TAY, F.Cu at (291.0, 279.7)
- added L6: LSMGG160808T331RG, myparts:IND_LSMG_160808_TAY, F.Cu at (289.5, 252.0)
- added MT10: MountingHole_Pad, MountingHole:MountingHole_3.2mm_M3_Pad_TopBottom, F.Cu at (110.0, 295.0)
- added MT7: MountingHole_Pad, MountingHole:MountingHole_3.2mm_M3_Pad_TopBottom, F.Cu at (80.0, 145.0)
- added MT8: MountingHole_Pad, MountingHole:MountingHole_3.2mm_M3_Pad_TopBottom, F.Cu at (110.0, 145.0)
- added MT9: MountingHole_Pad, MountingHole:MountingHole_3.2mm_M3_Pad_TopBottom, F.Cu at (80.0, 295.0)
- added R10: 4.99K, Resistor_SMD:R_0402_1005Metric, F.Cu at (262.7, 137.5)
- added R11: 11.4K, Resistor_SMD:R_0402_1005Metric, F.Cu at (281.5, 187.5)
- added R12: 1.0K, Resistor_SMD:R_0402_1005Metric, F.Cu at (281.5, 190.0)
- added R13: 100, Resistor_SMD:R_0402_1005Metric, F.Cu at (268.5, 205.0)
- added R14: KRL6432E-M-R010-F-T1, myparts:RES_6432_SUS, F.Cu at (273.0, 204.0)
- added R15: 100, Resistor_SMD:R_0402_1005Metric, F.Cu at (267.5, 181.5)
- added R16: 100, Resistor_SMD:R_0402_1005Metric, F.Cu at (268.5, 203.0)
- added R17: 0.01, myparts:RES_6432_SUS, F.Cu at (272.4, 182.5)
- added R18: 100, Resistor_SMD:R_0402_1005Metric, F.Cu at (267.5, 183.5)
- added R19: 4.99K, Resistor_SMD:R_0402_1005Metric, F.Cu at (263.1, 207.5)
- added R20: 4.99K, Resistor_SMD:R_0402_1005Metric, F.Cu at (263.0, 186.0)
- added R21: 0, Resistor_SMD:R_0402_1005Metric, F.Cu at (286.3, 261.7)
- added R22: 53K, Resistor_SMD:R_0402_1005Metric, F.Cu at (279.7, 261.2)
- added R23: 0, Resistor_SMD:R_0402_1005Metric, F.Cu at (285.7, 288.3)
- added R24: 33.2K, Resistor_SMD:R_0402_1005Metric, F.Cu at (280.2, 289.3)
- added R25: 0, Resistor_SMD:R_0402_1005Metric, F.Cu at (285.2, 312.2)
- added R26: 18.0K, Resistor_SMD:R_0402_1005Metric, F.Cu at (279.7, 313.2)
- added R27: 0, Resistor_SMD:R_0402_1005Metric, F.Cu at (285.3, 300.2)
- added R28: 24.9K, Resistor_SMD:R_0402_1005Metric, F.Cu at (279.8, 301.2)
- added R29: 0, Resistor_SMD:R_0402_1005Metric, F.Cu at (285.7, 276.7)
- added R30: 49.9K, Resistor_SMD:R_0402_1005Metric, F.Cu at (280.2, 277.7)
- added R31: 4.99K, Resistor_SMD:R_0402_1005Metric, F.Cu at (266.6, 277.3)
- added R32: KRL2012E-M-R220-F-T5, myparts:RESC1220X70N, F.Cu at (276.7, 314.6)
- added R33: KRL2012E-M-R220-F-T5, myparts:RESC1220X70N, F.Cu at (276.7, 249.3)
- added R34: KRL2012E-M-R220-F-T5, myparts:RESC1220X70N, F.Cu at (276.8, 302.6)
- added R35: KRL2012E-M-R220-F-T5, myparts:RESC1220X70N, F.Cu at (277.2, 279.1)
- added R36: KRL2012E-M-R220-F-T5, myparts:RESC1220X70N, F.Cu at (277.2, 290.7)
- added R37: 11.4K, Resistor_SMD:R_0402_1005Metric, F.Cu at (279.7, 250.0)
- added R38: 1.0K, Resistor_SMD:R_0402_1005Metric, F.Cu at (279.7, 247.7)
- added R4: KRL6432E-M-R010-F-T1, myparts:RES_6432_SUS, F.Cu at (272.6, 155.5)
- added R40: 4.99K, Resistor_SMD:R_0402_1005Metric, F.Cu at (272.1, 227.3)
- added R41: 9K, Resistor_SMD:R_0402_1005Metric, F.Cu at (281.5, 233.3)
- added R42: 1K, Resistor_SMD:R_0402_1005Metric, F.Cu at (279.5, 233.3)
- added R43: 9K, Resistor_SMD:R_0402_1005Metric, F.Cu at (281.6, 232.3)
- added R44: 1K, Resistor_SMD:R_0402_1005Metric, F.Cu at (279.6, 232.3)
- added R45: 9K, Resistor_SMD:R_0402_1005Metric, F.Cu at (281.6, 231.3)
- added R46: 1K, Resistor_SMD:R_0402_1005Metric, F.Cu at (279.6, 231.3)
- added R47: 9.56K, Resistor_SMD:R_0402_1005Metric, F.Cu at (279.6, 230.3)
- added R48: 9K, Resistor_SMD:R_0402_1005Metric, F.Cu at (281.6, 230.3)
- added R49: 9.56K, Resistor_SMD:R_0402_1005Metric, F.Cu at (279.6, 229.3)
- added R5: 100, Resistor_SMD:R_0402_1005Metric, F.Cu at (267.1, 133.0)
- added R50: 9K, Resistor_SMD:R_0402_1005Metric, F.Cu at (281.6, 229.3)
- added R51: 9.56K, Resistor_SMD:R_0402_1005Metric, F.Cu at (279.6, 228.3)
- added R52: 9K, Resistor_SMD:R_0402_1005Metric, F.Cu at (281.6, 228.3)
- added R53: KRL2012E-M-R220-F-T5, myparts:RESC1220X70N, F.Cu at (276.7, 262.1)
- added R6: 100, Resistor_SMD:R_0402_1005Metric, F.Cu at (268.1, 154.5)
- added R7: 0.01, myparts:RES_6432_SUS, F.Cu at (272.1, 134.0)
- added R8: 100, Resistor_SMD:R_0402_1005Metric, F.Cu at (267.1, 135.0)
- added R9: 4.99K, Resistor_SMD:R_0402_1005Metric, F.Cu at (262.8, 159.0)
- added U1: ~, myparts:burden, F.Cu at (94.0, 126.0)
- added U10: LT3045xDD, Package_DFN_QFN:DFN-10-1EP_3x3mm_P0.5mm_EP1.65x2.38mm, F.Cu at (282.8, 263.7)
- added U11: LT3045xDD, Package_DFN_QFN:DFN-10-1EP_3x3mm_P0.5mm_EP1.65x2.38mm, F.Cu at (283.1, 291.3)
- added U12: LT3045xDD, Package_DFN_QFN:DFN-10-1EP_3x3mm_P0.5mm_EP1.65x2.38mm, F.Cu at (282.7, 315.2)
- added U13: LT3045xDD, Package_DFN_QFN:DFN-10-1EP_3x3mm_P0.5mm_EP1.65x2.38mm, F.Cu at (282.8, 303.2)
- added U14: LT3045xDD, Package_DFN_QFN:DFN-10-1EP_3x3mm_P0.5mm_EP1.65x2.38mm, F.Cu at (283.2, 279.7)
- added U15: LTC2991CMS_TRPBF, myparts:MSOP-16_MS, F.Cu at (261.4, 230.6)
- added U16: LTC2991CMS_TRPBF, myparts:MSOP-16_MS, F.Cu at (261.8, 277.5)
- added U17: 3-641215-6, myparts:3-641215-6_TYC, F.Cu at (291.8, 226.0)
- added U18: LTC2991CMS_TRPBF, myparts:MSOP-16_MS, F.Cu at (272.7, 230.6)
- added U19: LT3015EDDPBF, myparts:DFN-8_DD, F.Cu at (282.7, 251.7)
- added U2: LT1963AEQ, Package_TO_SOT_SMD:TO-263-5_TabPin3, F.Cu at (293.1, 133.0)
- added U3: LT3015xQ-15, Package_TO_SOT_SMD:TO-263-5_TabPin3, F.Cu at (293.1, 153.0)
- added U4: LT6105, Package_TO_SOT_SMD:SOT-23-5, F.Cu at (263.3, 155.6)
- added U5: LT6105, Package_TO_SOT_SMD:SOT-23-5, F.Cu at (263.2, 134.4)
- added U6: LT1963AEQ, Package_TO_SOT_SMD:TO-263-5_TabPin3, F.Cu at (293.5, 181.5)
- added U7: LT3015xQ-15, Package_TO_SOT_SMD:TO-263-5_TabPin3, F.Cu at (293.5, 201.5)
- added U8: LT6105, Package_TO_SOT_SMD:SOT-23-5, F.Cu at (263.6, 204.1)
- added U9: LT6105, Package_TO_SOT_SMD:SOT-23-5, F.Cu at (263.6, 182.9)
- C1: value C_Small -> 100uF; footprint Capacitor_SMD:C_0402_1005Metric -> myparts:CAP_EEFK_D8_PAN
- J5: value 39301022 -> 0836149012; footprint myparts:MOLEX_39301022 -> myparts:0836149012
- J7: value 0836149012 -> 61083-061402LF; footprint myparts:0836149012 -> myparts:AMPHENOL_61083-061402LF
- J8: value 0836149012 -> 1731130154; footprint myparts:0836149012 -> myparts:CONN_F15-26P135G0-5979_MOL
- R1: value R_Small_US -> 11.4K
- R2: value R_US -> 1.0K
- R3: value R_US -> 100
- moved J7 220.1 mm to (96.0, 286.0), turned to 0 degrees
- moved J5 183.6 mm to (94.0, 95.9), turned to 180 degrees
- moved J8 133.7 mm to (285.6, 100.3), turned to 0 degrees
- moved MT5 109.1 mm to (299.9, 329.9)
- moved J1 109.1 mm to (243.0, 321.3)
- moved J2 109.1 mm to (166.8, 321.3)
- moved J3 109.1 mm to (217.6, 321.3)
- moved MT1 109.1 mm to (68.8, 329.9)
- moved MT2 109.1 mm to (112.0, 329.9)
- moved MT3 109.1 mm to (250.6, 329.9)
- moved MT4 43.8 mm to (300.0, 110.0)
- moved MT6 43.7 mm to (68.8, 110.0)
- moved R3 33.0 mm to (268.1, 156.5), turned to 180 degrees
- moved R2 32.4 mm to (281.1, 141.5), turned to -90 degrees
- moved R1 32.2 mm to (281.1, 139.0), turned to -90 degrees
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- renumbered J6 to J1, J3 to J2, J4 to J3
Connections:
- C1 pad 1: Net-(C1-Pad1) -> +18V
- J1 pad A1: unconnected-(J6-PadA1) -> /channel/digio.out0
- J1 pad A2: unconnected-(J6-PadA2) -> /channel/digio.in0
- J1 pad B1: unconnected-(J6-PadB1) -> /channel/digio.out1
- J1 pad B2: unconnected-(J6-PadB2) -> /channel/digio.in1
- J1 pad C1: unconnected-(J6-PadC1) -> /channel/digio.out2
- J1 pad C2: unconnected-(J6-PadC2) -> /channel/digio.in2
- J1 pad D1: unconnected-(J6-PadD1) -> /channel/digio.out3
- J1 pad D2: unconnected-(J6-PadD2) -> /channel/digio.in3
- J5 pad 1: unconnected-(J5-Pad1) -> /channel/reg_out+
- J7 pad 1: unconnected-(J7-Pad1) -> /channel/digio.out0
- J7 pad 10: unconnected-(J7-Pad10) -> +1.8V
- J7 pad 11: unconnected-(J7-Pad11) -> /channel/digio.in1
- J7 pad 12: unconnected-(J7-Pad12) -> GND
- J7 pad 13: unconnected-(J7-Pad13) -> /channel/digio.in2
- J7 pad 14: unconnected-(J7-Pad14) -> GND
- J7 pad 15: unconnected-(J7-Pad15) -> /channel/digio.in3
- J7 pad 16: unconnected-(J7-Pad16) -> GND
- J7 pad 17: unconnected-(J7-Pad17) -> GND
- J7 pad 18: unconnected-(J7-Pad18) -> GND
- J7 pad 19: unconnected-(J7-Pad19) -> /channel/dac_sclk
- J7 pad 2: unconnected-(J7-Pad2) -> GND
- J7 pad 20: unconnected-(J7-Pad20) -> GND
- J7 pad 21: unconnected-(J7-Pad21) -> /channel/dac_sdin
- J7 pad 22: unconnected-(J7-Pad22) -> +3.3V
- J7 pad 23: unconnected-(J7-Pad23) -> /channel/dac_syncn
- J7 pad 24: unconnected-(J7-Pad24) -> +3.3V
- J7 pad 25: unconnected-(J7-Pad25) -> GND
- J7 pad 26: (no net) -> +3.3V
- J7 pad 27: (no net) -> /channel/mon_reset
- J7 pad 3: unconnected-(J7-Pad3) -> /channel/digio.out1
- J7 pad 4: unconnected-(J7-Pad4) -> GND
- J7 pad 5: unconnected-(J7-Pad5) -> /channel/digio.out2
- J7 pad 6: unconnected-(J7-Pad6) -> +1.8V
- J7 pad 7: unconnected-(J7-Pad7) -> /channel/digio.out3
- J7 pad 8: unconnected-(J7-Pad8) -> +1.8V
- J7 pad 9: unconnected-(J7-Pad9) -> /channel/digio.in0
- J8 pad 1: unconnected-(J8-Pad1) -> +15V_DCCT
- J8 pad 10: unconnected-(J8-Pad10) -> GND
- J8 pad 11: unconnected-(J8-Pad11) -> /channel/Iin0-
- J8 pad 12: unconnected-(J8-Pad12) -> /channel/Iin1-
- J8 pad 13: unconnected-(J8-Pad13) -> /dcct connector/Iout3-
- J8 pad 14: unconnected-(J8-Pad14) -> /dcct connector/fault34
- J8 pad 15: unconnected-(J8-Pad15) -> /dcct connector/Iout7-
- J8 pad 16: unconnected-(J8-Pad16) -> /dcct connector/Iout6-
- J8 pad 17: unconnected-(J8-Pad17) -> /dcct connector/Iout5-
- J8 pad 18: unconnected-(J8-Pad18) -> GND
- J8 pad 19: unconnected-(J8-Pad19) -> -15V_DCCT
- J8 pad 2: unconnected-(J8-Pad2) -> /channel/Iin0+
- J8 pad 20: unconnected-(J8-Pad20) -> /dcct connector/Iout4+
- J8 pad 21: unconnected-(J8-Pad21) -> /dcct connector/Iout4-
- J8 pad 22: unconnected-(J8-Pad22) -> /dcct connector/fault56
- J8 pad 23: unconnected-(J8-Pad23) -> /dcct connector/fault78
- J8 pad 24: unconnected-(J8-Pad24) -> /dcct connector/Iout8+
- J8 pad 25: unconnected-(J8-Pad25) -> /dcct connector/Iout8-
- J8 pad 26: (no net) -> -15V_DCCT
- J8 pad 3: unconnected-(J8-Pad3) -> /channel/Iin1+
- J8 pad 4: unconnected-(J8-Pad4) -> /dcct connector/Iout3+
- J8 pad 5: unconnected-(J8-Pad5) -> /dcct connector/fault12
- J8 pad 6: unconnected-(J8-Pad6) -> /dcct connector/Iout7+
- J8 pad 7: unconnected-(J8-Pad7) -> /dcct connector/Iout6+
- J8 pad 8: unconnected-(J8-Pad8) -> /dcct connector/Iout5+
- J8 pad 9: unconnected-(J8-Pad9) -> +15V_DCCT
- R1 pad 1: Net-(D1-K) -> /regulators/+15v -15v DCCT Regulators/+15V_DCCT_REG
- R1 pad 2: Net-(C1-Pad1) -> Net-(U2-ADJ)
- R2 pad 1: Net-(D1-K) -> Net-(U2-ADJ)
- R2 pad 2: Net-(C1-Pad1) -> GND
- R3 pad 1: Net-(D1-K) -> /regulators/+15v -15v DCCT Regulators/-15V_DCCT_REG
- R3 pad 2: Net-(C1-Pad1) -> Net-(U4--)
Other:
- board size 241.3 x 171.4 mm -> 241.3 x 248.9 mm

Commit message: Add all 4 channels
Parts:
- removed the J5 at (94.0, 95.9)
- removed the U1 at (94.0, 126.0)
- added J10: 0836149012, myparts:0836149012, F.Cu at (140.0, 95.0)
- added J11: 61083-061402LF, myparts:AMPHENOL_61083-061402LF, F.Cu at (185.0, 155.0)
- added J12: 61083-061402LF, myparts:AMPHENOL_61083-061402LF, F.Cu at (186.6, 282.8)
- added J13: 0836149012, myparts:0836149012, F.Cu at (185.0, 95.0)
- added J14: 61083-061402LF, myparts:AMPHENOL_61083-061402LF, F.Cu at (230.0, 155.0)
- added J15: 61083-061402LF, myparts:AMPHENOL_61083-061402LF, F.Cu at (230.0, 285.0)
- added J16: 0836149012, myparts:0836149012, F.Cu at (230.0, 95.0)
- added J7: 0836149012, myparts:0836149012, F.Cu at (95.0, 95.0)
- added J8: 61083-061402LF, myparts:AMPHENOL_61083-061402LF, F.Cu at (140.0, 155.0)
- added J9: 61083-061402LF, myparts:AMPHENOL_61083-061402LF, F.Cu at (140.0, 285.0)
- added MT11: MountingHole_Pad, MountingHole:MountingHole_3.2mm_M3_Pad_TopBottom, F.Cu at (125.0, 145.0)
- added MT12: MountingHole_Pad, MountingHole:MountingHole_3.2mm_M3_Pad_TopBottom, F.Cu at (155.0, 145.0)
- added MT13: MountingHole_Pad, MountingHole:MountingHole_3.2mm_M3_Pad_TopBottom, F.Cu at (125.1, 295.0)
- added MT14: MountingHole_Pad, MountingHole:MountingHole_3.2mm_M3_Pad_TopBottom, F.Cu at (155.0, 295.0)
- added MT15: MountingHole_Pad, MountingHole:MountingHole_3.2mm_M3_Pad_TopBottom, F.Cu at (170.0, 145.0)
- added MT16: MountingHole_Pad, MountingHole:MountingHole_3.2mm_M3_Pad_TopBottom, F.Cu at (200.0, 145.0)
- added MT17: MountingHole_Pad, MountingHole:MountingHole_3.2mm_M3_Pad_TopBottom, F.Cu at (170.0, 295.0)
- added MT18: MountingHole_Pad, MountingHole:MountingHole_3.2mm_M3_Pad_TopBottom, F.Cu at (200.0, 295.0)
- added MT19: MountingHole_Pad, MountingHole:MountingHole_3.2mm_M3_Pad_TopBottom, F.Cu at (215.0, 145.0)
- added MT20: MountingHole_Pad, MountingHole:MountingHole_3.2mm_M3_Pad_TopBottom, F.Cu at (245.0, 145.0)
- added MT21: MountingHole_Pad, MountingHole:MountingHole_3.2mm_M3_Pad_TopBottom, F.Cu at (214.9, 295.0)
- added MT22: MountingHole_Pad, MountingHole:MountingHole_3.2mm_M3_Pad_TopBottom, F.Cu at (245.0, 295.0)
- added U19: ~, myparts:burden, F.Cu at (95.0, 120.0)
- added U20: ~, myparts:burden, F.Cu at (140.0, 120.0)
- added U21: ~, myparts:burden, F.Cu at (185.0, 120.0)
- added U22: ~, myparts:burden, F.Cu at (230.0, 120.0)
- moved J4 2.00 mm to (95.0, 155.0)
- moved J6 1.42 mm to (285.0, 99.0)
- moved J5 1.41 mm to (95.0, 285.0)
- moved C43 0.22 mm to (293.0, 292.0)
- moved C45 0.22 mm to (286.5, 291.8)
- moved C46 0.22 mm to (280.0, 293.8)
- moved C47 0.22 mm to (278.5, 294.1)
- moved C48 0.22 mm to (276.5, 294.8)
- moved C56 0.22 mm to (287.8, 303.9)
- moved L4 0.22 mm to (290.3, 315.2)
- moved L6 0.22 mm to (290.8, 279.7)
- moved R27 0.22 mm to (285.5, 288.3)
- moved R28 0.22 mm to (280.0, 289.3)
- moved R29 0.22 mm to (277.0, 290.7)
- moved U13 0.22 mm to (282.4, 315.2)
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- renumbered C65 to C31, C31 to C32, C63 to C33, C64 to C34, C32 to C35, C33 to C36, C66 to C37, C34 to C38, C67 to C39, C35 to C40, C68 to C41, C36 to C42, C37 to C43, C38 to C44, C39 to C45, C40 to C46, C41 to C47, C42 to C48, C43 to C49, C44 to C50, C45 to C51, C46 to C52, C47 to C53, C48 to C54, C49 to C55, C50 to C56, C51 to C57, C52 to C58, C53 to C59, C54 to C60, C55 to C61, C56 to C62, C57 to C63, C58 to C64, C59 to C65, C60 to C66, C61 to C67, C62 to C68, J3 to J1, J1 to J3, J6 to J4, J7 to J5, J8 to J6, L6 to L1, L1 to L2, L2 to L3, L3 to L4, L4 to L5, L5 to L6, R33 to R23, R53 to R24, R37 to R25, R38 to R26, R23 to R27, R24 to R28, R36 to R29, R25 to R30, R26 to R31, R27 to R33, R28 to R34, R34 to R35, R29 to R36, R30 to R37, R35 to R38, R41 to R39, R42 to R40, R43 to R41, R44 to R42, R45 to R43, R46 to R44, R47 to R45, R48 to R46, R49 to R47, R50 to R48, R51 to R49, R52 to R50, R31 to R51, R40 to R52, U17 to U1, U19 to U10, U10 to U11, U11 to U12, U12 to U13, U13 to U14, U14 to U15, U18 to U17, U15 to U18
Connections:
- net /channel/digin_rtn renamed /Ch1 Daughterboard/digin.rtn
- net /channel/digout_rtn renamed /Ch1 Daughterboard/digout.rtn
- net /dcct connector/fault12 renamed /DCCT connector/flt.12
- net /dcct connector/fault34 renamed /DCCT connector/flt.34
- net /dcct connector/fault56 renamed /DCCT connector/flt.56
- net /dcct connector/fault78 renamed /DCCT connector/flt.78
- J1 pad A1: unconnected-(J3-PadA1) -> /Ch4 Daughterboard/dcct.cnv
- J1 pad A10: unconnected-(J3-PadA10) -> /Ch3 Daughterboard/digio.in0
- J1 pad A2: unconnected-(J3-PadA2) -> /Ch4 Daughterboard/dcct.sdo1
- J1 pad A3: unconnected-(J3-PadA3) (its old number) -> /Ch4 Daughterboard/dac.syncn
- J1 pad A4: unconnected-(J3-PadA4) -> /Ch4 Daughterboard/digio.out2
- J1 pad A5: unconnected-(J3-PadA5) (its old number) -> /Ch4 Daughterboard/digio.in2
- J1 pad A7: unconnected-(J3-PadA7) (its old number) -> /Ch3 Daughterboard/dcct.sck
- J1 pad A8: unconnected-(J3-PadA8) -> /Ch3 Daughterboard/dac.sclk
- J1 pad A9: unconnected-(J3-PadA9) (its old number) -> /Ch3 Daughterboard/digio.out0
- J1 pad B1: unconnected-(J3-PadB1) -> /Ch4 Daughterboard/dcct.busy
- J1 pad B10: unconnected-(J3-PadB10) -> /Ch3 Daughterboard/digio.in1
- J1 pad B4: unconnected-(J3-PadB4) -> /Ch4 Daughterboard/digio.out3
- J1 pad B5: unconnected-(J3-PadB5) -> /Ch4 Daughterboard/digio.in3
- J1 pad B7: unconnected-(J3-PadB7) -> /Ch3 Daughterboard/dcct.sdo0
- J1 pad B8: unconnected-(J3-PadB8) -> /Ch3 Daughterboard/dac.sdin
- J1 pad B9: unconnected-(J3-PadB9) -> /Ch3 Daughterboard/digio.out1
- J1 pad C1: unconnected-(J3-PadC1) -> /Ch4 Daughterboard/dcct.sck
- J1 pad C10: unconnected-(J3-PadC10) -> /Ch3 Daughterboard/digio.in2
- J1 pad C2: unconnected-(J3-PadC2) -> /Ch4 Daughterboard/dac.sclk
- J1 pad C3: unconnected-(J3-PadC3) -> /Ch4 Daughterboard/digio.out0
- J1 pad C4: unconnected-(J3-PadC4) -> /Ch4 Daughterboard/digio.in0
- J1 pad C6: unconnected-(J3-PadC6) -> /Ch3 Daughterboard/dcct.cnv
- J1 pad C7: unconnected-(J3-PadC7) -> /Ch3 Daughterboard/dcct.sdo1
- J1 pad C8: unconnected-(J3-PadC8) -> /Ch3 Daughterboard/dac.syncn
- J1 pad C9: unconnected-(J3-PadC9) -> /Ch3 Daughterboard/digio.out2
- J1 pad D1: unconnected-(J3-PadD1) -> /Ch4 Daughterboard/dcct.sdo0
- J1 pad D10: unconnected-(J3-PadD10) (its old number) -> /Ch3 Daughterboard/digio.in3
- J1 pad D2: unconnected-(J3-PadD2) -> /Ch4 Daughterboard/dac.sdin
- J1 pad D3: unconnected-(J3-PadD3) -> /Ch4 Daughterboard/digio.out1
- J1 pad D4: unconnected-(J3-PadD4) (its old number) -> /Ch4 Daughterboard/digio.in1
- J1 pad D6: unconnected-(J3-PadD6) (its old number) -> /Ch3 Daughterboard/dcct.busy
- J1 pad D9: unconnected-(J3-PadD9) -> /Ch3 Daughterboard/digio.out3
- J2 pad A1: unconnected-(J2-PadA1) -> /Ch2 Daughterboard/dcct.cnv
- J2 pad A10: unconnected-(J2-PadA10) -> /Ch1 Daughterboard/digio.in0
- J2 pad A2: unconnected-(J2-PadA2) -> /Ch2 Daughterboard/dcct.sdo1
- J2 pad A3: unconnected-(J2-PadA3) -> /Ch2 Daughterboard/dac.syncn
- J2 pad A4: unconnected-(J2-PadA4) -> /Ch2 Daughterboard/digio.out2
- J2 pad A5: unconnected-(J2-PadA5) -> /Ch2 Daughterboard/digio.in2
- J2 pad A7: unconnected-(J2-PadA7) -> /Ch1 Daughterboard/dcct.sck
- J2 pad A8: unconnected-(J2-PadA8) -> /Ch1 Daughterboard/dac.sclk
- J2 pad A9: unconnected-(J2-PadA9) -> /Ch1 Daughterboard/digio.out0
- J2 pad B1: unconnected-(J2-PadB1) -> /Ch2 Daughterboard/dcct.busy
- J2 pad B10: unconnected-(J2-PadB10) -> /Ch1 Daughterboard/digio.in1
- J2 pad B4: unconnected-(J2-PadB4) -> /Ch2 Daughterboard/digio.out3
- J2 pad B5: unconnected-(J2-PadB5) -> /Ch2 Daughterboard/digio.in3
- J2 pad B7: unconnected-(J2-PadB7) -> /Ch1 Daughterboard/dcct.sdo0
- J2 pad B8: unconnected-(J2-PadB8) -> /Ch1 Daughterboard/dac.sdin
- J2 pad B9: unconnected-(J2-PadB9) -> /Ch1 Daughterboard/digio.out1
- J2 pad C1: unconnected-(J2-PadC1) -> /Ch2 Daughterboard/dcct.sck
- J2 pad C10: unconnected-(J2-PadC10) -> /Ch1 Daughterboard/digio.in2
- J2 pad C2: unconnected-(J2-PadC2) -> /Ch2 Daughterboard/dac.sclk
- J2 pad C3: unconnected-(J2-PadC3) -> /Ch2 Daughterboard/digio.out0
- J2 pad C4: unconnected-(J2-PadC4) -> /Ch2 Daughterboard/digio.in0
- J2 pad C6: unconnected-(J2-PadC6) -> /Ch1 Daughterboard/dcct.cnv
- J2 pad C7: unconnected-(J2-PadC7) -> /Ch1 Daughterboard/dcct.sdo1
- J2 pad C8: unconnected-(J2-PadC8) -> /Ch1 Daughterboard/dac.syncn
- J2 pad C9: unconnected-(J2-PadC9) -> /Ch1 Daughterboard/digio.out2
- J2 pad D1: unconnected-(J2-PadD1) -> /Ch2 Daughterboard/dcct.sdo0
- J2 pad D10: unconnected-(J2-PadD10) -> /Ch1 Daughterboard/digio.in3
- J2 pad D2: unconnected-(J2-PadD2) -> /Ch2 Daughterboard/dac.sdin
- J2 pad D3: unconnected-(J2-PadD3) -> /Ch2 Daughterboard/digio.out1
- J2 pad D4: unconnected-(J2-PadD4) -> /Ch2 Daughterboard/digio.in1
- J2 pad D6: unconnected-(J2-PadD6) -> /Ch1 Daughterboard/dcct.busy
- J2 pad D9: unconnected-(J2-PadD9) -> /Ch1 Daughterboard/digio.out3
- J3 pad A1: /channel/digio.out0 -> unconnected-(J3-PadA1)
- J3 pad A10: unconnected-(J1-PadA10) -> /Ch1 Daughterboard/mon.fs
- J3 pad A2: /channel/digio.in0 -> unconnected-(J3-PadA2)
- J3 pad A4: unconnected-(J1-PadA4) -> /Ch4 Daughterboard/mon.fs
- J3 pad A6: unconnected-(J1-PadA6) (its old number) -> /Ch3 Daughterboard/mon.fs
- J3 pad A8: unconnected-(J1-PadA8) -> /Ch2 Daughterboard/mon.fs
- J3 pad B1: /channel/digio.out1 -> unconnected-(J3-PadB1)
- J3 pad B10: unconnected-(J1-PadB10) -> /Ch1 Daughterboard/mon.sdo
- J3 pad B2: /channel/digio.in1 -> unconnected-(J3-PadB2)
- J3 pad B3: unconnected-(J1-PadB3) (its old number) -> /Ch4 Daughterboard/mon.reset
- J3 pad B4: unconnected-(J1-PadB4) -> /Ch4 Daughterboard/mon.sdo
- J3 pad B5: unconnected-(J1-PadB5) -> /Ch3 Daughterboard/mon.reset
- J3 pad B6: unconnected-(J1-PadB6) (its old number) -> /Ch3 Daughterboard/mon.sdo
- J3 pad B7: unconnected-(J1-PadB7) -> /Ch2 Daughterboard/mon.reset
- J3 pad B8: unconnected-(J1-PadB8) -> /Ch2 Daughterboard/mon.sdo
- J3 pad B9: unconnected-(J1-PadB9) -> /Ch1 Daughterboard/mon.reset
- J3 pad C1: /channel/digio.out2 -> unconnected-(J3-PadC1)
- J3 pad C10: unconnected-(J1-PadC10) -> /Ch1 Daughterboard/mon.sclk
- J3 pad C2: /channel/digio.in2 -> unconnected-(J3-PadC2)
- J3 pad C3: unconnected-(J1-PadC3) -> /Ch4 Daughterboard/mon.cnvrt
- J3 pad C4: unconnected-(J1-PadC4) -> /Ch4 Daughterboard/mon.sclk
- J3 pad C5: unconnected-(J1-PadC5) (its old number) -> /Ch3 Daughterboard/mon.cnvrt
- J3 pad C6: unconnected-(J1-PadC6) -> /Ch3 Daughterboard/mon.sclk
- J3 pad C7: unconnected-(J1-PadC7) -> /Ch2 Daughterboard/mon.cnvrt
- J3 pad C8: unconnected-(J1-PadC8) -> /Ch2 Daughterboard/mon.sclk
- J3 pad C9: unconnected-(J1-PadC9) -> /Ch1 Daughterboard/mon.cnvrt
- J3 pad D1: /channel/digio.out3 -> unconnected-(J3-PadD1)
- J3 pad D2: /channel/digio.in3 -> unconnected-(J3-PadD2)
- J3 pad D3: unconnected-(J1-PadD3) -> /Ch4 Daughterboard/mon.busy
- J3 pad D5: unconnected-(J1-PadD5) (its old number) -> /Ch3 Daughterboard/mon.busy
- J3 pad D7: unconnected-(J1-PadD7) (its old number) -> /Ch2 Daughterboard/mon.busy
- J3 pad D9: unconnected-(J1-PadD9) -> /Ch1 Daughterboard/mon.busy
- J4 pad 10: /channel/digin_spare -> /Ch1 Daughterboard/digin.spare
- J4 pad 12: /channel/digin_flt2 -> /Ch1 Daughterboard/digin.flt2
- J4 pad 14: /channel/digin_flt1 -> /Ch1 Daughterboard/digin.flt1
- J4 pad 16: /channel/digin_acon -> /Ch1 Daughterboard/digin.acon
- J4 pad 2: /channel/digout_spare -> /Ch1 Daughterboard/digout.spare
- J4 pad 20: /channel/ps_spare- -> /Ch1 Daughterboard/ps.spare-
- J4 pad 22: /channel/ps_spare+ -> /Ch1 Daughterboard/ps.spare+
- J4 pad 26: /channel/ps_ignd- -> /Ch1 Daughterboard/ps.ignd-
- J4 pad 28: /channel/ps_ignd+ -> /Ch1 Daughterboard/ps.ignd+
- J4 pad 32: /channel/ps_vout- -> /Ch1 Daughterboard/ps.vout-
- J4 pad 34: /channel/ps_vout+ -> /Ch1 Daughterboard/ps.vout+
- J4 pad 4: /channel/digout_reset -> /Ch1 Daughterboard/digout.reset
- J4 pad 40: /channel/reg_out- -> /Ch1 Daughterboard/reg.out-
- J4 pad 42: /channel/reg_out+ -> /Ch1 Daughterboard/reg.out+
- J4 pad 48: /channel/dcct0+ -> /Ch1 Burden Resistor/Vout0.dcct+
- J4 pad 50: /channel/dcct0- -> /Ch1 Burden Resistor/Vout0.dcct-
- J4 pad 56: /channel/dcct1+ -> /Ch1 Burden Resistor/Vout1.dcct+
- J4 pad 58: /channel/dcct1- -> /Ch1 Burden Resistor/Vout1.dcct-
- J4 pad 6: /channel/digout_on2 -> /Ch1 Daughterboard/digout.on2
- J4 pad 8: /channel/digout_on1 -> /Ch1 Daughterboard/digout.on1
- J5 pad 1: /channel/digio.out0 -> /Ch1 Daughterboard/digio.out0
- J5 pad 11: /channel/digio.in1 -> /Ch1 Daughterboard/digio.in1
- J5 pad 13: /channel/digio.in2 -> /Ch1 Daughterboard/digio.in2
- J5 pad 15: /channel/digio.in3 -> /Ch1 Daughterboard/digio.in3
- J5 pad 19: /channel/dac_sclk -> /Ch1 Daughterboard/dac.sclk
- J5 pad 21: /channel/dac_sdin -> /Ch1 Daughterboard/dac.sdin
- J5 pad 23: /channel/dac_syncn -> /Ch1 Daughterboard/dac.syncn
- J5 pad 27: /channel/mon_reset -> /Ch1 Daughterboard/mon.reset
- J5 pad 29: /channel/mon_convert -> /Ch1 Daughterboard/mon.cnvrt
- J5 pad 3: /channel/digio.out1 -> /Ch1 Daughterboard/digio.out1
- J5 pad 31: /channel/mon_busy -> /Ch1 Daughterboard/mon.busy
- J5 pad 33: /channel/mon_fs -> /Ch1 Daughterboard/mon.fs
- J5 pad 35: /channel/mon_sdo -> /Ch1 Daughterboard/mon.sdo
- J5 pad 37: /channel/mon_sclk -> /Ch1 Daughterboard/mon.sclk
- J5 pad 41: /channel/dcct_cnv -> /Ch1 Daughterboard/dcct.cnv
- J5 pad 43: /channel/dcct_busy -> /Ch1 Daughterboard/dcct.busy
- J5 pad 45: /channel/dcct_sck -> /Ch1 Daughterboard/dcct.sck
- J5 pad 47: /channel/dcct0_sdo -> /Ch1 Daughterboard/dcct.sdo0
- J5 pad 49: /channel/dcct1_sdo -> /Ch1 Daughterboard/dcct.sdo1
- J5 pad 5: /channel/digio.out2 -> /Ch1 Daughterboard/digio.out2
- J5 pad 7: /channel/digio.out3 -> /Ch1 Daughterboard/digio.out3
- J5 pad 9: /channel/digio.in0 -> /Ch1 Daughterboard/digio.in0
- J6 pad 11: /channel/Iin0- -> /Ch1 Burden Resistor/Iin0.dcct-
- J6 pad 12: /channel/Iin1- -> /Ch1 Burden Resistor/Iin1.dcct-
- J6 pad 13: /dcct connector/Iout3- -> /Ch2 Burden Resistor/Iin0.dcct-
- J6 pad 15: /dcct connector/Iout7- -> /Ch4 Burden Resistor/Iin0.dcct-
- J6 pad 16: /dcct connector/Iout6- -> /Ch3 Burden Resistor/Iin1.dcct-
- J6 pad 17: /dcct connector/Iout5- -> /Ch3 Burden Resistor/Iin0.dcct-
- J6 pad 2: /channel/Iin0+ -> /Ch1 Burden Resistor/Iin0.dcct+
- J6 pad 20: /dcct connector/Iout4+ -> /Ch2 Burden Resistor/Iin1.dcct+
- J6 pad 21: /dcct connector/Iout4- -> /Ch2 Burden Resistor/Iin1.dcct-
- J6 pad 24: /dcct connector/Iout8+ -> /Ch4 Burden Resistor/Iin1.dcct+
- J6 pad 25: /dcct connector/Iout8- -> /Ch4 Burden Resistor/Iin1.dcct-
- J6 pad 3: /channel/Iin1+ -> /Ch1 Burden Resistor/Iin1.dcct+
- J6 pad 4: /dcct connector/Iout3+ -> /Ch2 Burden Resistor/Iin0.dcct+
- J6 pad 6: /dcct connector/Iout7+ -> /Ch4 Burden Resistor/Iin0.dcct+
- J6 pad 7: /dcct connector/Iout6+ -> /Ch3 Burden Resistor/Iin1.dcct+
- J6 pad 8: /dcct connector/Iout5+ -> /Ch3 Burden Resistor/Iin0.dcct+
