File: psc_carrier_brd.kicad_pcb (KiCad board)
At the start: 2 copper layers, 241.3 x 248.9 mm, 187 parts, among them J1 6469028-1, J10 0836149012, J11 61083-061402LF, J12 61083-061402LF, J13 0836149012, J14 61083-061402LF, J15 61083-061402LF, J16 0836149012, J2 6469028-1, J3 6469028-1, J4 61083-061402LF, J5 61083-061402LF, J6 1731130154, J7 0836149012, J8 61083-061402LF, J9 61083-061402LF, U1 3-641215-6, U10 LT3015EDDPBF, U11 LT3045xDD, U12 LT3045xDD, U13 LT3045xDD, U14 LT3045xDD, U15 LT3045xDD, U16 LTC2991CMS_TRPBF, U17 LTC2991CMS_TRPBF, U18 LTC2991CMS_TRPBF, U2 LT1963AEQ, U3 LT3015xQ-15, U4 LT6105, U5 LT6105, U6 LT1963AEQ, U7 LT3015xQ-15, U8 LT6105, U9 LT6105

Commit message: Start routing
Parts:
- removed the C1 at (270.7, 126.0)
- removed the C10 at (281.1, 161.5)
- removed the C11 at (277.1, 139.3)
- removed the C12 at (261.6, 131.5)
- removed the C13 at (264.2, 158.5)
- removed the C14 at (261.7, 152.5)
- removed the C15 at (279.1, 139.1)
- removed the C2 at (271.1, 147.5)
- removed the C3 at (279.1, 125.8)
- removed the C4 at (279.4, 145.5)
- removed the C5 at (295.7, 127.4)
- removed the C6 at (281.1, 146.1)
- removed the C7 at (270.5, 162.0)
- removed the C8 at (270.6, 140.5)
- removed the C9 at (279.1, 161.8)
- removed the R1 at (281.1, 139.0)
- removed the R10 at (262.7, 137.5)
- removed the R2 at (281.1, 141.5)
- removed the R3 at (268.1, 156.5)
- removed the R36 at (285.5, 276.7)
- removed the R37 at (280.0, 277.7)
- removed the R38 at (277.0, 279.1)
- removed the R4 at (272.6, 155.5)
- removed the R5 at (267.1, 133.0)
- removed the R6 at (268.1, 154.5)
- removed the R7 at (272.1, 134.0)
- removed the R8 at (267.1, 135.0)
- removed the R9 at (262.8, 159.0)
- removed the U15 at (282.9, 279.7)
- removed the U2 at (293.1, 133.0)
- removed the U3 at (293.1, 153.0)
- removed the U4 at (263.3, 155.6)
- removed the U5 at (263.2, 134.4)
- added C46: 0.022u, Capacitor_SMD:C_0603_1608Metric, F.Cu at (293.0, 276.5)
- added C47: 10u, Capacitor_SMD:C_0603_1608Metric, F.Cu at (286.5, 283.5)
- added C48: 10p, Capacitor_SMD:C_0603_1608Metric, F.Cu at (291.5, 276.5)
- added C49: 10u, Capacitor_SMD:C_0603_1608Metric, F.Cu at (295.5, 283.5)
- added C50: 330p, Capacitor_SMD:C_0603_1608Metric, F.Cu at (290.0, 274.0)
- added C51: 1u, Capacitor_SMD:C_0603_1608Metric, F.Cu at (285.0, 280.0)
- added C52: 10p, Capacitor_SMD:C_0603_1608Metric, F.Cu at (287.7, 277.3)
- added C53: 22u, Capacitor_SMD:C_0805_2012Metric, F.Cu at (295.5, 300.9)
- added C54: 22u, Capacitor_SMD:C_0805_2012Metric, F.Cu at (292.5, 300.8)
- added C55: 22u, Capacitor_SMD:C_0805_2012Metric, F.Cu at (289.5, 300.8)
- added C56: 22u, Capacitor_SMD:C_0805_2012Metric, F.Cu at (286.5, 300.8)
- added C60: 100uF, myparts:CAP_EEFK_D8_PAN, F.Cu at (271.9, 143.5)
- added C67: 100uF, myparts:CAPMP7.6X4.3_4.3N_KEM, F.Cu at (271.5, 158.5)
- added C68: 10uF, Capacitor_SMD:C_0603_1608Metric, F.Cu at (278.7, 184.0)
- added C69: 0.1uF, Capacitor_SMD:C_0402_1005Metric, F.Cu at (278.5, 182.0)
- added C70: 10uF, Capacitor_SMD:C_0603_1608Metric, F.Cu at (278.2, 160.4)
- added C71: 0.1uF, Capacitor_SMD:C_0402_1005Metric, F.Cu at (277.7, 158.5)
- added C72: 0.1uF, Capacitor_SMD:C_0402_1005Metric, B.Cu at (260.5, 174.0)
- added C73: 0.1uF, Capacitor_SMD:C_0402_1005Metric, B.Cu at (260.5, 176.0)
- added C74: 0.1uF, Capacitor_SMD:C_0402_1005Metric, B.Cu at (259.0, 152.5)
- added C75: 0.1uF, Capacitor_SMD:C_0402_1005Metric, F.Cu at (278.9, 245.3)
- added D1: GREEN, LED_SMD:LED_0603_1608Metric, F.Cu at (300.8, 277.8)
- added J4: 39301022, myparts:MOLEX_39301022, F.Cu at (293.6, 312.0)
- added Q1: NX7002BKW, Package_TO_SOT_SMD:SOT-323_SC-70, F.Cu at (301.0, 274.7)
- added R26: 41.2k, Resistor_SMD:R_0402_1005Metric, F.Cu at (295.5, 278.8)
- added R27: 1k, Resistor_SMD:R_0402_1005Metric, F.Cu at (298.1, 275.3)
- added R28: 8.45k, Resistor_SMD:R_0402_1005Metric, F.Cu at (290.0, 276.8)
- added R29: 10.2k, Resistor_SMD:R_0402_1005Metric, F.Cu at (295.5, 280.8)
- added R30: 1.13k, Resistor_SMD:R_0402_1005Metric, F.Cu at (295.5, 279.8)
- added R31: 4.7k, Resistor_SMD:R_0402_1005Metric, F.Cu at (282.0, 280.3)
- added R32: 4.7k, Resistor_SMD:R_0402_1005Metric, F.Cu at (283.5, 278.0)
- added R33: 0, Resistor_SMD:R_0402_1005Metric, F.Cu at (283.5, 280.3)
- added R34: 42.2k, Resistor_SMD:R_0402_1005Metric, F.Cu at (288.0, 278.8)
- added R35: 10.2k, Resistor_SMD:R_0402_1005Metric, F.Cu at (288.0, 275.8)
- added R50: 11.4K, Resistor_SMD:R_0402_1005Metric, F.Cu at (281.5, 157.0)
- added R51: 1.0K, Resistor_SMD:R_0402_1005Metric, F.Cu at (281.5, 159.0)
- added R52: 100, Resistor_SMD:R_0402_1005Metric, F.Cu at (268.5, 172.5)
- added R53: KRL6432E-M-R010-F-T1, myparts:RES_6432_SUS, F.Cu at (273.4, 173.5)
- added R54: 100, Resistor_SMD:R_0402_1005Metric, F.Cu at (269.0, 150.5)
- added R55: 100, Resistor_SMD:R_0402_1005Metric, F.Cu at (268.5, 176.5)
- added R56: KRL6432E-M-R010-F-T1, myparts:RES_6432_SUS, F.Cu at (273.6, 151.5)
- added R57: 100, Resistor_SMD:R_0402_1005Metric, F.Cu at (269.0, 154.5)
- added R58: 4.99K, Resistor_SMD:R_0402_1005Metric, F.Cu at (263.5, 171.5)
- added R59: 4.99K, Resistor_SMD:R_0402_1005Metric, F.Cu at (260.0, 150.5)
- added R60: 10K, Resistor_SMD:R_0402_1005Metric, F.Cu at (276.0, 238.5)
- added R61: 10K, Resistor_SMD:R_0402_1005Metric, F.Cu at (276.0, 240.5)
- added R62: 10K, Resistor_SMD:R_0402_1005Metric, F.Cu at (276.0, 242.5)
- added R63: 10K, Resistor_SMD:R_0402_1005Metric, F.Cu at (276.0, 244.5)
- added R64: 10K, Resistor_SMD:R_0402_1005Metric, F.Cu at (276.0, 246.5)
- added R65: 10K, Resistor_SMD:R_0402_1005Metric, F.Cu at (276.0, 248.5)
- added R66: 10K, Resistor_SMD:R_0402_1005Metric, F.Cu at (276.0, 250.5)
- added R67: 10K, Resistor_SMD:R_0402_1005Metric, F.Cu at (276.0, 252.4)
- added R68: 10K, Resistor_SMD:R_0402_1005Metric, F.Cu at (269.0, 256.0)
- added R69: 10K, Resistor_SMD:R_0402_1005Metric, F.Cu at (269.0, 258.0)
- added TP1: Net-(Q1-G), TestPoint:TestPoint_THTPad_D2.0mm_Drill1.0mm, F.Cu at (298.5, 270.8)
- added TP2: +5.0V, TestPoint:TestPoint_THTPad_D2.0mm_Drill1.0mm, F.Cu at (301.5, 301.3)
- added U11: LT8643S, myparts:QFN-24-4EP_4x4mm_P0.5mm_EP1.125x1.125mm, F.Cu at (290.8, 282.6)
- added U19: LT1963AEQ, Package_TO_SOT_SMD:TO-263-5_TabPin3, F.Cu at (293.1, 150.7)
- added U20: LT3015xQ-15, Package_TO_SOT_SMD:TO-263-5_TabPin3, F.Cu at (292.6, 169.3)
- added U21: LT6105, Package_TO_SOT_SMD:SOT-23-5, F.Cu at (264.6, 174.6)
- added U22: LT6105, Package_TO_SOT_SMD:SOT-23-5, F.Cu at (263.6, 152.6)
- added U23: CD74HC4050, myparts:PW16, F.Cu at (282.0, 240.9)
- C61: value 10uF -> 100uF; footprint Capacitor_SMD:C_0603_1608Metric -> myparts:CAP_EEFK_D8_PAN
- C63: value 0.1uF -> 10uF; footprint Capacitor_SMD:C_0402_1005Metric -> Capacitor_SMD:C_0603_1608Metric
- C65: value 10uF -> 0.1uF; footprint Capacitor_SMD:C_0603_1608Metric -> Capacitor_SMD:C_0402_1005Metric
- C66: footprint Capacitor_SMD:C_1206_3216Metric -> myparts:CAPMP7.6X4.3_4.3N_KEM
- L6: value LSMGG160808T331RG -> 2.2u; footprint myparts:IND_LSMG_160808_TAY -> myparts:COILCRAFT_MSS1048
- moved C64 139.8 mm to (286.0, 142.5), turned to 0 degrees
- moved C62 138.4 mm to (282.5, 142.2), turned to 0 degrees
- moved C61 116.8 mm to (272.0, 165.5), turned to 0 degrees
- moved C65 105.6 mm to (282.1, 177.0), turned to 0 degrees
- moved C66 103.4 mm to (271.5, 180.0), turned to 0 degrees
- moved C63 100.3 mm to (282.3, 180.0), turned to 0 degrees
- moved U12 33.8 mm to (248.8, 308.7)
- moved C58 33.8 mm to (250.6, 305.6)
- moved R48 33.8 mm to (253.6, 308.6)
- moved U1 23.0 mm to (297.5, 248.3)
- moved R49 22.4 mm to (260.5, 246.5)
- moved U13 22.4 mm to (261.2, 249.7)
- moved R36 21.7 mm to (270.5, 252.0)
- moved R37 21.7 mm to (268.5, 252.0)
- moved R38 21.7 mm to (270.5, 251.0)
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- renumbered C16 to C1, C25 to C10, C26 to C11, C27 to C12, C28 to C13, C29 to C14, C30 to C15, C31 to C16, C32 to C17, C33 to C18, C34 to C19, C17 to C2, C35 to C20, C36 to C21, C37 to C22, C38 to C23, C39 to C24, C40 to C25, C41 to C26, C42 to C27, C43 to C28, C44 to C29, C18 to C3, C45 to C30, C46 to C31, C47 to C32, C48 to C33, C49 to C34, C50 to C35, C51 to C36, C52 to C37, C53 to C38, C54 to C39, C19 to C4, C55 to C40, C56 to C41, C57 to C42, C58 to C43, C59 to C44, C60 to C45, C20 to C5, C67 to C57, C68 to C58, C69 to C59, C21 to C6, C22 to C7, C23 to C8, C24 to C9, J9 to J10, J10 to J11, J11 to J12, J12 to J13, J13 to J14, J14 to J15, J15 to J16, J16 to J17, J4 to J5, J5 to J6, J6 to J7, J7 to J8, J8 to J9, R11 to R1, R20 to R10, R21 to R11, R22 to R12, R23 to R13, R24 to R14, R25 to R15, R26 to R16, R27 to R17, R28 to R18, R29 to R19, R12 to R2, R30 to R20, R31 to R21, R32 to R22, R33 to R23, R34 to R24, R35 to R25, R13 to R3, R39 to R36, R40 to R37, R41 to R38, R42 to R39, R14 to R4, R43 to R40, R44 to R41, R45 to R42, R46 to R43, R47 to R44, R48 to R45, R49 to R46, R50 to R47, R51 to R48, R52 to R49, R15 to R5, R16 to R6, R17 to R7, R18 to R8, R19 to R9, U14 to U10, U16 to U12, U17 to U13, U18 to U14, U19 to U15, U20 to U16, U21 to U17, U22 to U18, U6 to U2, U7 to U3, U8 to U4, U9 to U5, U10 to U6, U11 to U7, U12 to U8, U13 to U9
Connections:
- net /regulators/+15v -15v PSC Regulators/+15V_DCCT_REG renamed /regulators/+15v -15v PSC Regulators/+15V_PSC_REG
- net /regulators/+15v -15v PSC Regulators/-15V_DCCT_REG renamed /regulators/+15v -15v PSC Regulators/-15V_PSC_REG
- C17 pad 1: +6V -> +15V
- C28 pad 1: +6V -> +5.0V
- C34 pad 1: +6V -> +5.0V
- C40 pad 1: +6V -> +5.0V
- C61 pad 1: +6V -> -18V
- C62 pad 1: Net-(U15-EN/UV) -> +18V
- C63 pad 1: Net-(U15-EN/UV) -> -18V
- C64 pad 1: /regulators/+5VD regulator/imon_hi -> +18V
- C65 pad 1: /regulators/+5VD regulator/imon_hi -> -18V
- C66 pad 1: /regulators/+5VD regulator/imon_hi -> /regulators/+15v -15v DCCT Regulators/-15V_DCCT_REG
- J12 pad 1: /Ch3 Daughterboard/digout.rtn -> /Ch3 Daughterboard/digin.rtn
- J12 pad 11: /Ch3 Daughterboard/digin.rtn -> /Ch3 Daughterboard/digout.rtn
- J12 pad 13: /Ch3 Daughterboard/digin.rtn -> /Ch3 Daughterboard/digout.rtn
- J12 pad 15: /Ch3 Daughterboard/digin.rtn -> /Ch3 Daughterboard/digout.rtn
- J12 pad 3: /Ch3 Daughterboard/digout.rtn -> /Ch3 Daughterboard/digin.rtn
- J12 pad 5: /Ch3 Daughterboard/digout.rtn -> /Ch3 Daughterboard/digin.rtn
- J12 pad 7: /Ch3 Daughterboard/digout.rtn -> /Ch3 Daughterboard/digin.rtn
- J12 pad 9: /Ch3 Daughterboard/digin.rtn -> /Ch3 Daughterboard/digout.rtn
- J15 pad 1: /Ch4 Daughterboard/digout.rtn -> /Ch4 Daughterboard/digin.rtn
- J15 pad 11: /Ch4 Daughterboard/digin.rtn -> /Ch4 Daughterboard/digout.rtn
- J15 pad 13: /Ch4 Daughterboard/digin.rtn -> /Ch4 Daughterboard/digout.rtn
- J15 pad 15: /Ch4 Daughterboard/digin.rtn -> /Ch4 Daughterboard/digout.rtn
- J15 pad 3: /Ch4 Daughterboard/digout.rtn -> /Ch4 Daughterboard/digin.rtn
- J15 pad 5: /Ch4 Daughterboard/digout.rtn -> /Ch4 Daughterboard/digin.rtn
- J15 pad 7: /Ch4 Daughterboard/digout.rtn -> /Ch4 Daughterboard/digin.rtn
- J15 pad 9: /Ch4 Daughterboard/digin.rtn -> /Ch4 Daughterboard/digout.rtn
- J3 pad A1: unconnected-(J3-PadA1) -> /DCCT Fault Logic/dcct_flt_buf.12
- J3 pad A10: /Ch1 Daughterboard/mon.fs -> unconnected-(J3-PadA10)
- J3 pad A3: unconnected-(J3-PadA3) -> /Ch4 Daughterboard/mon.busy
- J3 pad A4: /Ch4 Daughterboard/mon.fs -> unconnected-(J3-PadA4)
- J3 pad A5: unconnected-(J3-PadA5) -> /Ch3 Daughterboard/mon.busy
- J3 pad A6: /Ch3 Daughterboard/mon.fs -> unconnected-(J3-PadA6)
- J3 pad A7: unconnected-(J3-PadA7) -> /Ch2 Daughterboard/mon.busy
- J3 pad A8: /Ch2 Daughterboard/mon.fs -> unconnected-(J3-PadA8)
- J3 pad A9: unconnected-(J3-PadA9) -> /Ch1 Daughterboard/mon.busy
- J3 pad B1: unconnected-(J3-PadB1) -> /DCCT Fault Logic/dcct_flt_buf.34
- J3 pad B10: /Ch1 Daughterboard/mon.sdo -> unconnected-(J3-PadB10)
- J3 pad B3: /Ch4 Daughterboard/mon.reset -> /Ch4 Daughterboard/mon.fs
- J3 pad B4: /Ch4 Daughterboard/mon.sdo -> unconnected-(J3-PadB4)
- J3 pad B5: /Ch3 Daughterboard/mon.reset -> /Ch3 Daughterboard/mon.fs
- J3 pad B6: /Ch3 Daughterboard/mon.sdo -> unconnected-(J3-PadB6)
- J3 pad B7: /Ch2 Daughterboard/mon.reset -> /Ch2 Daughterboard/mon.fs
- J3 pad B8: /Ch2 Daughterboard/mon.sdo -> unconnected-(J3-PadB8)
- J3 pad B9: /Ch1 Daughterboard/mon.reset -> /Ch1 Daughterboard/mon.fs
- J3 pad C1: unconnected-(J3-PadC1) -> /DCCT Fault Logic/dcct_flt_buf.56
- J3 pad C10: /Ch1 Daughterboard/mon.sclk -> /regulators/i2c_sda
- J3 pad C2: unconnected-(J3-PadC2) -> /Ch4 Daughterboard/mon.reset
- J3 pad C3: /Ch4 Daughterboard/mon.cnvrt -> /Ch4 Daughterboard/mon.sdo
- J3 pad C4: /Ch4 Daughterboard/mon.sclk -> /Ch3 Daughterboard/mon.reset
- J3 pad C5: /Ch3 Daughterboard/mon.cnvrt -> /Ch3 Daughterboard/mon.sdo
- J3 pad C6: /Ch3 Daughterboard/mon.sclk -> /Ch2 Daughterboard/mon.reset
- J3 pad C7: /Ch2 Daughterboard/mon.cnvrt -> /Ch2 Daughterboard/mon.sdo
- J3 pad C8: /Ch2 Daughterboard/mon.sclk -> /Ch1 Daughterboard/mon.reset
- J3 pad C9: /Ch1 Daughterboard/mon.cnvrt -> /Ch1 Daughterboard/mon.sdo
- J3 pad D1: unconnected-(J3-PadD1) -> /DCCT Fault Logic/dcct_flt_buf.78
- J3 pad D10: unconnected-(J3-PadD10) -> /regulators/i2c_scl
- J3 pad D2: unconnected-(J3-PadD2) -> /Ch4 Daughterboard/mon.cnvrt
- J3 pad D3: /Ch4 Daughterboard/mon.busy -> /Ch4 Daughterboard/mon.sclk
- J3 pad D4: unconnected-(J3-PadD4) -> /Ch3 Daughterboard/mon.cnvrt
- J3 pad D5: /Ch3 Daughterboard/mon.busy -> /Ch3 Daughterboard/mon.sclk
- J3 pad D6: unconnected-(J3-PadD6) -> /Ch2 Daughterboard/mon.cnvrt
- J3 pad D7: /Ch2 Daughterboard/mon.busy -> /Ch2 Daughterboard/mon.sclk
- J3 pad D8: unconnected-(J3-PadD8) -> /Ch1 Daughterboard/mon.cnvrt
- J3 pad D9: /Ch1 Daughterboard/mon.busy -> /Ch1 Daughterboard/mon.sclk
- J5 pad 1: /Ch1 Daughterboard/digout.rtn -> /Ch1 Daughterboard/digin.rtn
- J5 pad 11: /Ch1 Daughterboard/digin.rtn -> /Ch1 Daughterboard/digout.rtn
- J5 pad 13: /Ch1 Daughterboard/digin.rtn -> /Ch1 Daughterboard/digout.rtn
- J5 pad 15: /Ch1 Daughterboard/digin.rtn -> /Ch1 Daughterboard/digout.rtn
- J5 pad 3: /Ch1 Daughterboard/digout.rtn -> /Ch1 Daughterboard/digin.rtn
- J5 pad 5: /Ch1 Daughterboard/digout.rtn -> /Ch1 Daughterboard/digin.rtn
- J5 pad 7: /Ch1 Daughterboard/digout.rtn -> /Ch1 Daughterboard/digin.rtn
- J5 pad 9: /Ch1 Daughterboard/digin.rtn -> /Ch1 Daughterboard/digout.rtn
- J7 pad 14: /DCCT connector/flt.34 -> /DCCT Fault Logic/dcct_flt.34
- J7 pad 22: /DCCT connector/flt.56 -> /DCCT Fault Logic/dcct_flt.56
- J7 pad 23: /DCCT connector/flt.78 -> /DCCT Fault Logic/dcct_flt.78
- J7 pad 5: /DCCT connector/flt.12 -> /DCCT Fault Logic/dcct_flt.12
- J9 pad 1: /Ch2 Daughterboard/digout.rtn -> /Ch2 Daughterboard/digin.rtn
- J9 pad 11: /Ch2 Daughterboard/digin.rtn -> /Ch2 Daughterboard/digout.rtn
- J9 pad 13: /Ch2 Daughterboard/digin.rtn -> /Ch2 Daughterboard/digout.rtn
- J9 pad 15: /Ch2 Daughterboard/digin.rtn -> /Ch2 Daughterboard/digout.rtn
- J9 pad 3: /Ch2 Daughterboard/digout.rtn -> /Ch2 Daughterboard/digin.rtn
- J9 pad 5: /Ch2 Daughterboard/digout.rtn -> /Ch2 Daughterboard/digin.rtn
- J9 pad 7: /Ch2 Daughterboard/digout.rtn -> /Ch2 Daughterboard/digin.rtn
- J9 pad 9: /Ch2 Daughterboard/digin.rtn -> /Ch2 Daughterboard/digout.rtn
- L2 pad 2: +6V -> +15V
- L3 pad 2: +6V -> +5.0V
- L4 pad 2: +6V -> +5.0V
- L5 pad 2: +6V -> +5.0V
- L6 pad 1: Net-(U15-EN/UV) -> Net-(L6-Pad1)
- L6 pad 2: +6V -> +5.0V
- R4 pad 1: -15V_DCCT -> -15V
- R6 pad 1: -15V_DCCT -> -15V
- R7 pad 1: +15V_DCCT -> +15V
- R8 pad 1: +15V_DCCT -> +15V
- U1 pad 5: +6.0V -> GND
- U12 pad 1: /regulators/+5VD regulator/imon_hi -> unconnected-(U12-V1-Pad1)
- U12 pad 2: +5V -> unconnected-(U12-V2-Pad2)
Routing:
- net GND: track 0.00 -> 269.4 mm, vias 0 -> 133
- net /Ch1 Burden Resistor/Iin0.dcct+: track 0.00 -> 222.9 mm
- net /Ch1 Burden Resistor/Iin0.dcct-: track 0.00 -> 203.0 mm
- net /Ch1 Daughterboard/mon.reset: track 0.00 -> 172.6 mm, vias 0 -> 3
- net /Ch1 Daughterboard/mon.fs: track 0.00 -> 171.4 mm, vias 0 -> 3
- net /Ch1 Daughterboard/mon.cnvrt: track 0.00 -> 170.0 mm, vias 0 -> 3
- net /Ch1 Daughterboard/mon.busy: track 0.00 -> 169.9 mm, vias 0 -> 3
- net /Ch1 Daughterboard/mon.sdo: track 0.00 -> 165.6 mm, vias 0 -> 3
- net /Ch1 Daughterboard/mon.sclk: track 0.00 -> 163.8 mm, vias 0 -> 3
- net /Ch2 Burden Resistor/Iin0.dcct+: track 0.00 -> 158.6 mm, vias 0 -> 1
- net /Ch2 Burden Resistor/Iin0.dcct-: track 0.00 -> 138.7 mm, vias 0 -> 1
- net /Ch2 Daughterboard/mon.reset: track 0.00 -> 130.9 mm, vias 0 -> 3
- net /Ch2 Daughterboard/mon.cnvrt: track 0.00 -> 129.7 mm, vias 0 -> 3
- net /Ch2 Daughterboard/mon.busy: track 0.00 -> 128.9 mm, vias 0 -> 3
- net /Ch2 Daughterboard/mon.fs: track 0.00 -> 128.8 mm, vias 0 -> 3
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Other:
- copper layers 2 -> 10

Commit message: Change board size length to 255mm
Other:
- board size 241.3 x 248.9 mm -> 241.3 x 255 mm
Changed lines of the file:
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@@
 	)
 	(gr_line
-		(start 63.7 86.08)
-		(end 305 86.08)
+		(start 63.7 80)
+		(end 305 80)
 		(stroke
 			(width 0.05)
@@
 	)
 	(gr_line
-		(start 305 86.08)
+		(start 305 80)
 		(end 305 335)
 		(stroke
@@
 	(gr_line
 		(start 63.7 335)
-		(end 63.7 86.08)
+		(end 63.7 80)
 		(stroke
 			(width 0.05)
