File: 5v_power_supply.kicad_sch (KiCad schematic)
At the start: 27 parts, among them Q1 NX7002BKW, U11 LT8643S

Commit message: Start routing
Parts:
- removed R33: 0, Resistor_SMD:R_0402_1005Metric, symbol Device:R_Small_US
- removed U11: LT8643S, myparts:QFN-24-4EP_4x4mm_P0.5mm_EP1.125x1.125mm, symbol psc:LT8643S
- added R884: 10.2k, Resistor_SMD:R_0603_1608Metric, symbol Device:R_Small_US
- added R885: 1.13k, Resistor_SMD:R_0603_1608Metric, symbol Device:R_Small_US
- added U178: LT8643S, handmade:QFN-24-4EP_4x4mm_P0.5mm_EP1.125x1.125mm, symbol custom:LT8643S
- L22: renamed from L6; footprint myparts:COILCRAFT_MSS1048 -> handmade:COILCRAFT_MSS1048
- R875: renamed from R32; footprint Resistor_SMD:R_0402_1005Metric -> Resistor_SMD:R_0603_1608Metric; now fitted
- R876: renamed from R27; footprint Resistor_SMD:R_0402_1005Metric -> Resistor_SMD:R_0603_1608Metric
- R877: renamed from R26; footprint Resistor_SMD:R_0402_1005Metric -> Resistor_SMD:R_0603_1608Metric
- R878: renamed from R29; footprint Resistor_SMD:R_0402_1005Metric -> Resistor_SMD:R_0603_1608Metric
- R879: renamed from R30; footprint Resistor_SMD:R_0402_1005Metric -> Resistor_SMD:R_0603_1608Metric
- R880: renamed from R28; footprint Resistor_SMD:R_0402_1005Metric -> Resistor_SMD:R_0603_1608Metric
- R881: renamed from R31; footprint Resistor_SMD:R_0402_1005Metric -> Resistor_SMD:R_0603_1608Metric
- R882: renamed from R34; footprint Resistor_SMD:R_0402_1005Metric -> Resistor_SMD:R_0603_1608Metric
- R883: renamed from R35; footprint Resistor_SMD:R_0402_1005Metric -> Resistor_SMD:R_0603_1608Metric; MFG (none) -> Stackpole Electronics Inc; MFG_PN (none) -> RMCF0603FT10K2
- renumbered C46 to C808, C47 to C809, C49 to C810, C48 to C811, C50 to C812, C51 to C813, C52 to C814, C53 to C815, C54 to C816, C55 to C817, C56 to C818, D1 to D140, Q1 to Q90, TP1 to TP35, TP2 to TP36
Connections:
- net GND: now also R885.2, U178.16 (GND), U178.25 (EPAD), U178.26 (EPAD), U178.27 (EPAD), U178.28 (EPAD), U178.3 (GND)
- net at L22.1: now also U178.10 (SW), U178.11 (SW), U178.12 (SW), U178.8 (SW), U178.9 (SW)
- net at R878.2, R879.1: now also U178.17 (EN/UV)
- net at R877.1: now also U178.18 (RT)
- net at C813.1, R881.2: now also U178.2 (INTVCC)
- net 5V_PSCLK: now reaches R875.1
- net 5V_PSCLK: now also U178.20 (SYNC/MODE)
- net at C808.1: now also U178.21 (TR/SS)
- net at C811.1, R880.1: now also U178.22 (VC)
- net 5V_PG: now reaches Q90.1 (G), R881.1, TP35.1
- net 5V_PG: now also U178.23 (PG)
- net at C814.2, R882.2, R883.1: now also U178.24 (FB)
- net +18V renamed +12V
- net +12V: now also U178.13 (VIN), U178.14 (VIN), U178.5 (VIN), U178.6 (VIN)
- net +5.0V renamed 5V
- net 5V: now also R884.1, U178.1 (BIAS)
- new net 5V_VMEAS: R884.2, R885.1
Other:
- note removed: "SYNC PIN GND = Burst Mode (Low Output Load, lowest noise) Float = Forced Continuous Mode INTVCC = Spread spectrum mode"
- title: (none) -> RHIC MADC2\nSCHEMATIC DRAWING
- moved on the sheet: C808, C809, C810, C811, C812, C813, C814, C815, C816, C817, C818, D140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
