File: burden.kicad_sch (KiCad schematic)
At the start: 1 part

Commit message: Start routing
Parts:
- renumbered U19 to U15
Changed lines of the file:
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@@
 		(on_board yes)
 		(dnp no)
-		(property "Reference" "U19"
+		(property "Reference" "U15"
 			(at 151.13 109.982 0)
 			(effects
@@
 			(project "psc_carrier_brd"
 				(path "/40891cc8-bf64-41f4-8f69-a607d7b280eb/06895ba2-0dba-4ca0-bd23-a9fa74452504"
-					(reference "U21")
+					(reference "U17")
 					(unit 1)
 				)
 				(path "/40891cc8-bf64-41f4-8f69-a607d7b280eb/34ed6f92-cccc-48eb-b305-3dcd35c3cab7"
-					(reference "U22")
+					(reference "U18")
 					(unit 1)
 				)
 				(path "/40891cc8-bf64-41f4-8f69-a607d7b280eb/9ce9c2c4-cc81-44b8-8079-482e57213d61"
-					(reference "U19")
+					(reference "U15")
 					(unit 1)
 				)
 				(path "/40891cc8-bf64-41f4-8f69-a607d7b280eb/9ed33170-dc63-4493-90d5-5a0ea9d80229"
-					(reference "U20")
+					(reference "U16")
 					(unit 1)
 				)

Commit message: Finished layout
Parts:
- U15: value ~ -> Burden; MFG (none) -> BNL; MFG_PN (none) -> BNL
Changed lines of the file:
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@@
 			)
 		)
-		(property "Value" "~"
+		(property "Value" "Burden"
 			(at 150.495 73.66 0)
 			(effects
@@
 					(size 1.27 1.27)
 				)
+				(hide yes)
 			)
 		)
@@
 			)
 		)
-		(property "Description" ""
+		(property "Description" "Burden Resistor Daughterboard"
 			(at 140.97 74.93 0)
 			(effects
+				(font
+					(size 1.27 1.27)
+				)
+				(hide yes)
+			)
+		)
+		(property "MFG" "BNL"
+			(at 140.97 74.93 0)
+			(effects
+				(font
+					(size 1.27 1.27)
+				)
+				(hide yes)
+			)
+		)
+		(property "MFG_PN" "BNL"
+			(at 140.97 74.93 0)
+			(effects
