File: dcct_fault.kicad_sch (KiCad schematic)
At the start: 10 parts, among them U23 CD74HC4050

Commit message: Finished layout
Parts:
- C75: Cost (none) -> .01; MFG (none) -> Taiyo Yuden; MFG_PN (none) -> TMK105BJ104KV-F
- R60, R61, R62, R63, R64, R65, R66, R67: Cost (none) -> 0.01; MFG (none) -> Panasonic; MFG_PN (none) -> ERJ-2RKF1002X
- U23: Cost (none) -> 0.37
Connections:
- net at R62.2, R66.1, U23.7 (Cin): no longer R67.1
- net at R63.2, U23.9 (Din): now also R67.1
