File: p5.0vd.kicad_sch (KiCad schematic)
At the start: 27 parts, among them Q1 NX7002BKW, U11 LT8643S

Commit message: Finished layout
Parts:
- C46: value 0.022u -> 0.022uF; Cost (none) -> 0.01; MFG Samsung Electro-Mechanics -> Samsung
- C47, C49: value 10u -> 10uF; Cost (none) -> .04; MFG Samsung Electro-Mechanics -> Samsung
- C48, C52: value 10p -> 10pF; Cost (none) -> .01; MFG Samsung Electro-Mechanics -> Samsung
- C50: value 330p -> 330pF; Cost (none) -> 0.01; MFG Samsung Electro-Mechanics -> Samsung
- C51: value 1u -> 1uF; Cost (none) -> 0.01; MFG Samsung Electro-Mechanics -> Samsung
- C53, C54, C55, C56: value 22u -> 22uF; Cost (none) -> 0.04; MFG Samsung Electro-Mechanics -> Samsung
- D1: Cost (none) -> 0.1
- L6: value 2.2u -> 2.2uF; Cost (none) -> 3.26
- Q1: Cost (none) -> 0.1; MFG Nexperia USA Inc. -> Nexperia
- R26: value 41.2k -> 41.2K; Cost (none) -> 0.01; MFG Stackpole Electronics Inc -> Panasonic; MFG_PN RMCF0603FT41K2 -> ERJ-2RKF4122X
- R27: value 1k -> 1.0K; Cost (none) -> 0.01; MFG Stackpole Electronics Inc -> Panasonic; MFG_PN RMCF0603FT1K00 -> ERJ-2RKF1001X
- R28: value 8.45k -> 8.45K; Cost (none) -> 0.01; MFG Stackpole Electronics Inc -> Panasonic; MFG_PN RMCF0603FT8K45 -> ERJ-2RKF8451X
- R29: value 10.2k -> 10.2K; Cost (none) -> 0.01; MFG Stackpole Electronics Inc -> Panasonic; MFG_PN RMCF0603FT10K2 -> ERJ-2RKF1022X
- R30: value 1.13k -> 1.13K; Cost (none) -> 0.01; MFG Stackpole Electronics Inc -> Panasonic; MFG_PN RMCF0603FT1K13 -> ERJ-2RKF1131X
- R31, R32: value 4.7k -> 4.7K; Cost (none) -> 0.01; MFG Stackpole Electronics Inc -> Panasonic; MFG_PN RMCF0603FT4K70 -> ERJ-2RKF4701X
- R33: Cost (none) -> 0.01; MFG Stackpole Electronics Inc -> Panasonic; MFG_PN RMCF0603FT4K70 -> ERJ-2GE0R00X
- R34: value 42.2k -> 42.2K; Cost (none) -> 0.01; MFG Stackpole Electronics Inc -> Panasonic; MFG_PN RMCF0603FT42K2 -> ERJ-2RKF4222X
- R35: value 10.2k -> 10.2K; Cost (none) -> 0.01; MFG (none) -> Panasonic; MFG_PN (none) -> ERJ-2RKF1022X
- TP1, TP2: MFG (none) -> N/A; MFG_PN (none) -> N/A; now not fitted
- U11: Cost (none) -> 9.56; MFG (none) -> Analog Devices; MFG_PN (none) -> LT8643SEV#PBF
Connections:
- net +5vrego: now reaches L6.1, U11.10 (SW), U11.11 (SW), U11.12 (SW), U11.8 (SW), U11.9 (SW)
Other:
- moved on the sheet: L6
