File: ps_conn.kicad_sch (KiCad schematic)
At the start: 1 part, among them J7 0836149012

Commit message: Start routing
Parts:
- renumbered J7 to J8
Connections:
- no-connect marks 0 -> 5
Changed lines of the file:
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@@
 		(color 0 0 0 0)
+	)
+	(no_connect
+		(at 120.65 100.33)
+	)
+	(no_connect
+		(at 135.89 101.6)
+	)
+	(no_connect
+		(at 120.65 118.11)
+	)
+	(no_connect
+		(at 120.65 90.17)
+	)
+	(no_connect
+		(at 135.89 91.44)
 	)
 	(bus_entry
@@
 		(dnp no)
 		(fields_autoplaced yes)
-		(property "Reference" "J7"
+		(property "Reference" "J8"
 			(at 128.27 76.2 0)
 			(effects
@@
 			(project "psc_carrier_brd"
 				(path "/40891cc8-bf64-41f4-8f69-a607d7b280eb/270c0463-7903-4545-8f56-97f30d2fa241"
-					(reference "J16")
+					(reference "J17")
 					(unit 1)
 				)
 				(path "/40891cc8-bf64-41f4-8f69-a607d7b280eb/507954ec-02e9-46c0-a919-b9e1fc42de5f"
-					(reference "J7")
+					(reference "J8")
 					(unit 1)
 				)
 				(path "/40891cc8-bf64-41f4-8f69-a607d7b280eb/81f88550-83e3-4fa8-bdcb-5b1e15f2b3a9"
-					(reference "J10")
+					(reference "J11")
 					(unit 1)
 				)
 				(path "/40891cc8-bf64-41f4-8f69-a607d7b280eb/f9b49ffc-0448-499b-a1fa-488e5d512990"
-					(reference "J13")
+					(reference "J14")
 					(unit 1)
 				)

Commit message: Finished layout
Parts:
- J8: Cost (none) -> 17.82; MFG (none) -> Molex; MFG_PN (none) -> 0836149012
Changed lines of the file:
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@@
 			)
 		)
-		(property "Description" ""
+		(property "Description" "CONN MICRO-D PLUG 25POS R/A SLDR"
 			(at 127 83.82 0)
 			(effects
+				(font
+					(size 1.27 1.27)
+				)
+				(hide yes)
+			)
+		)
+		(property "Cost" "17.82"
+			(at 127 83.82 0)
+			(effects
+				(font
+					(size 1.27 1.27)
+				)
+				(hide yes)
+			)
+		)
+		(property "MFG" "Molex"
+			(at 127 83.82 0)
+			(effects
+				(font
+					(size 1.27 1.27)
+				)
+				(hide yes)
+			)
+		)
+		(property "MFG_PN" "0836149012"
+			(at 127 83.82 0)
+			(effects
