File: psc_carrier_brd.kicad_sch (KiCad schematic)
At the start: 6 parts

Commit message: Start routing
Other:
- added sheet DCCT Fault Logic (dcct_fault.kicad_sch)
- sheet regulators ports: added i2c_scl, i2c_sda; removed none
- sheet zuDFE Connectors ports: added dcct_flt_buf{12 34 56 78}, i2c_scl, i2c_sda; removed none
Changed lines of the file:
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@@
+		)
+	)
+	(bus
+		(pts
+			(xy 62.23 243.84) (xy 83.82 243.84)
+		)
+		(stroke
+			(width 0)
+			(type default)
 		)
 	)
@@
 		)
 	)
+	(wire
+		(pts
+			(xy 260.35 125.73) (xy 313.69 125.73)
+		)
+		(stroke
+			(width 0)
+			(type default)
+		)
+	)
 	(bus
 		(pts
@@
 	(wire
 		(pts
+			(xy 260.35 128.27) (xy 313.69 128.27)
+		)
+		(stroke
+			(width 0)
+			(type default)
+		)
+	)
+	(wire
+		(pts
 			(xy 384.81 196.85) (xy 384.81 195.58)
 		)
@@
 		(pts
 			(xy 132.08 45.72) (xy 139.7 45.72)
+		)
+		(stroke
+			(width 0)
+			(type default)
+		)
+	)
+	(bus
+		(pts
+			(xy 195.58 243.84) (xy 220.98 243.84)
 		)
 		(stroke
@@
 			)
 		)
+		(pin "dcct_flt_buf{12 34 56 78}" input
+			(at 220.98 243.84 180)
+			(effects
+				(font
+					(size 1.27 1.27)
+				)
+				(justify left)
+			)
+		)
+		(pin "i2c_sda" input
+			(at 260.35 128.27 0)
+			(effects
+				(font
+					(size 1.27 1.27)
+				)
+				(justify right)
+			)
+		)
+		(pin "i2c_scl" input
+			(at 260.35 125.73 0)
+			(effects
+				(font
+					(size 1.27 1.27)
+				)
+				(justify right)
+			)
+		)
 		(instances
 			(project "psc_carrier_brd"
@@
 	)
 	(sheet
+		(at 83.82 238.76)
+		(size 111.76 11.43)
+		(exclude_from_sim no)
+		(in_bom yes)
+		(on_board yes)
+		(dnp no)
+		(fields_autoplaced yes)
+		(stroke
+			(width 0.1524)
+			(type solid)
+		)
+		(fill
+			(color 255 255 194 1.0000)
+		)
+		(property "Sheetname" "DCCT Fault Logic"
+			(at 83.82 238.0484 0)
+			(effects
+				(font
+					(size 1.27 1.27)
+				)
+				(justify left bottom)
+			)
+		)
+		(property "Sheetfile" "dcct_fault.kicad_sch"
+			(at 83.82 251.4096 0)
+			(effects
+				(font
+					(size 1.27 1.27)
+				)
+				(justify left top)
+			)
+		)
+		(pin "dcct_flt{12 34 56 78}" input
+			(at 83.82 243.84 180)
+			(effects
+				(font
+					(size 1.27 1.27)
+				)
+				(justify left)
+			)
+		)
+		(pin "dcct_flt_buf{12 34 56 78}" output
+			(at 195.58 243.84 0)
+			(effects
+				(font
+					(size 1.27 1.27)
+				)
+				(justify right)
+			)
+		)
+		(instances
+			(project "psc_carrier_brd"
+				(path "/40891cc8-bf64-41f4-8f69-a607d7b280eb"
+					(page "25")
+				)
+			)
+		)
+	)
+	(sheet
 		(at 82.55 40.64)
 		(size 49.53 7.62)
@@
 	)
 	(sheet
-		(at 331.47 127.635)
-		(size 53.975 45.085)
+		(at 313.69 113.03)
+		(size 54.61 45.72)
 		(exclude_from_sim no)
 		(in_bom yes)
@@
 		)
 		(property "Sheetname" "regulators"
-			(at 331.47 126.9234 0)
+			(at 313.69 112.3184 0)
 			(effects
 				(font
@@
 		)
 		(property "Sheetfile" "regs.kicad_sch"
-			(at 331.47 173.3046 0)
+			(at 313.69 158.6996 0)
 			(effects
 				(font
@@
 				)
 				(justify left top)
+			)
+		)
+		(pin "i2c_scl" input
+			(at 313.69 125.73 180)
+			(effects
+				(font
+					(size 1.27 1.27)
+				)
+				(justify left)
+			)
+		)
+		(pin "i2c_sda" input
+			(at 313.69 128.27 180)
+			(effects
+				(font
+					(size 1.27 1.27)
+				)
+				(justify left)
 			)
 		)
@@
 			)
 		)
-		(pin "flt{12 34 56 78}" input
+		(pin "flt{12 34 56 78}" output
 			(at 62.23 243.84 0)
 			(effects

Commit message: Finished layout
Parts:
- added MT23, MT24: MountingHole_Pad, MountingHole:MountingHole_4.3mm_M4_DIN965_Pad, symbol Mechanical:MountingHole_Pad
- added TP12, TP13, TP14, TP15, TP16, TP17: ${SHORT_NET_NAME(1)}, myparts:TestPoint_RCS-0C, symbol Connector:TestPoint
Connections:
- net GND: now also MT23.1, MT24.1, TP12.1, TP13.1, TP14.1, TP15.1, TP16.1, TP17.1
Other:
- sheet regulators ports: added enb; removed none
- sheet zuDFE Connectors ports: added enb; removed none
- note added: "zuPSC Carrier Board"
- moved on the sheet: MT1, MT2, MT3, MT4, MT5, MT6
