File: regs_15v.kicad_sch (KiCad schematic)
At the start: 29 parts, among them U2 LT1963AEQ, U3 LT3015xQ-15, U4 LT6105, U5 LT6105

Commit message: Finished layout
Parts:
- added TP8, TP9: ${SHORT_NET_NAME(1)}, TestPoint:TestPoint_THTPad_D2.0mm_Drill1.0mm, symbol Connector:TestPoint
- C1, C2: Cost (none) -> 0.44; MFG (none) -> Panasonic; MFG_PN (none) -> EEE-FTH101XAP
- C10, C12, C13, C14, C15, C5, C6: Cost (none) -> .01; MFG (none) -> Taiyo Yuden; MFG_PN (none) -> TMK105BJ104KV-F
- C11, C3, C4, C9: Cost (none) -> .04; MFG (none) -> Samsung; MFG_PN (none) -> CL10A106MA8NRNC
- C7, C8: Cost (none) -> 3.56; MFG (none) -> Kemet; MFG_PN (none) -> T521X107M025ATE060
- R1: value 11.4K -> 11.5K; Cost (none) -> 0.01; MFG (none) -> Panasonic; MFG_PN (none) -> ERJ-2RKF1152X
- R10, R9: Cost (none) -> 0.01; MFG (none) -> Panasonic; MFG_PN (none) -> ERJ-2RKF4991X
- R2: Cost (none) -> 0.01; MFG (none) -> Panasonic; MFG_PN (none) -> ERJ-2RKF1001X
- R3, R5, R6, R8: Cost (none) -> 0.01; MFG (none) -> Panasonic; MFG_PN (none) -> ERJ-2RKF1000X
- R4: value KRL6432E-M-R010-F-T1 -> 0.01; Cost (none) -> 0.71; MFG (none) -> Susumu; MFG_PN (none) -> KRL6432E-M-R010-F-T1
- R7: Cost (none) -> 0.71; MFG (none) -> Susumu; MFG_PN (none) -> KRL6432E-M-R010-F-T1
- U2: Cost (none) -> 5.57; MFG (none) -> Analog Devices; MFG_PN (none) -> LT1963AEQ#TRPBF
- U3: value LT3015xQ-15 -> LT3015EQ-15; Cost (none) -> 6.46; MFG (none) -> Analog Devices; MFG_PN (none) -> LT3015EQ-15#PBF
- U4, U5: value LT6105 -> LT6106; Cost (none) -> 2.01; MFG (none) -> Analog Devices; MFG_PN (none) -> LT6106CS5#TRMPBF
Connections:
- net +15V: now also TP8.1
- net -15V: now also TP9.1
- net -15V_PSC_REG: now also C7.2; no longer C7.1
- net -18V: now also C2.2; no longer C2.1
- net GND: now also C2.1, C7.1; no longer C2.2, C7.2
- net +5V renamed +5.0V
Other:
- moved on the sheet: C7
