File: regs_dcct_15v.kicad_sch (KiCad schematic)
At the start: 29 parts, among them U2 LT1963AEQ, U3 LT3015xQ-15, U4 LT6105, U5 LT6105

Commit message: Start routing
Parts:
- removed C1, C2: 100uF, myparts:CAP_EEFK_D8_PAN, symbol psc:EEE-FTH101XAP
- removed C10, C12, C13, C14, C15, C5, C6: 0.1uF, Capacitor_SMD:C_0402_1005Metric, symbol Device:C_Small
- removed C11, C3, C4, C9: 10uF, Capacitor_SMD:C_0603_1608Metric, symbol Device:C_Small
- removed C7, C8: 100uF, myparts:CAPMP7.6X4.3_4.3N_KEM, symbol psc:T521X107M025ATE060
- removed R1: 11.4K, Resistor_SMD:R_0402_1005Metric, symbol Device:R_US
- removed R10, R9: 4.99K, Resistor_SMD:R_0402_1005Metric, symbol Device:R_US
- removed R2: 1.0K, Resistor_SMD:R_0402_1005Metric, symbol Device:R_US
- removed R3, R5, R6, R8: 100, Resistor_SMD:R_0402_1005Metric, symbol Device:R_US
- removed R4: KRL6432E-M-R010-F-T1, myparts:RES_6432_SUS, symbol psc:KRL6432E-M-R010-F-T1
- removed R7: 0.01, myparts:RES_6432_SUS, symbol psc:KRL6432E-M-R010-F-T1
- removed U2: LT1963AEQ, Package_TO_SOT_SMD:TO-263-5_TabPin3, symbol Regulator_Linear:LT1963AEQ
- removed U3: LT3015xQ-15, Package_TO_SOT_SMD:TO-263-5_TabPin3, symbol Regulator_Linear:LT3015xQ-15
- removed U4, U5: LT6105, Package_TO_SOT_SMD:SOT-23-5, symbol psc:LT6105
- added C60, C61: 100uF, CAP_EEFK_D8_PAN, symbol psc:EEE-FTH101XAP
- added C62, C63, C68, C70: 10uF, Capacitor_SMD:C_0603_1608Metric, symbol Device:C_Small
- added C64, C65, C69, C71, C72, C73, C74: 0.1uF, Capacitor_SMD:C_0402_1005Metric, symbol Device:C_Small
- added C66, C67: 100uF, CAPMP7.6X4.3_4.3N_KEM, symbol psc:T521X107M025ATE060
- added R50: 11.4K, Resistor_SMD:R_0402_1005Metric, symbol Device:R_US
- added R51: 1.0K, Resistor_SMD:R_0402_1005Metric, symbol Device:R_US
- added R52, R54, R55, R57: 100, Resistor_SMD:R_0402_1005Metric, symbol Device:R_US
- added R53, R56: KRL6432E-M-R010-F-T1, myparts:RES_6432_SUS, symbol psc:KRL6432E-M-R010-F-T1
- added R58, R59: 4.99K, Resistor_SMD:R_0402_1005Metric, symbol Device:R_US
- added U19: LT1963AEQ, Package_TO_SOT_SMD:TO-263-5_TabPin3, symbol Regulator_Linear:LT1963AEQ
- added U20: LT3015xQ-15, Package_TO_SOT_SMD:TO-263-5_TabPin3, symbol Regulator_Linear:LT3015xQ-15
- added U21, U22: LT6105, Package_TO_SOT_SMD:SOT-23-5, symbol psc:LT6105
Connections:
- net +18V: now also C60.1, C62.1, C64.1, U19.1 (~{SHDN}), U19.2 (IN)
- net +5V: now also C73.1, U21.5 (V+)
- net -18V: now also C61.1, C63.1, C65.1, U20.1 (~{SHDN}), U20.3 (IN)
- net GND: now also C60.2, C61.2, C62.2, C63.2, C64.2, C65.2, C66.2, C67.2, C68.2, C69.2, C70.2, C71.2, C72.2, C73.2, C74.2, R51.2, R58.2, R59.2, U19.3 (GND), U20.2 (GND), U22.2 (V-)
- net isense_+15v: now also R59.1, U22.1
- net isense_-15v: now also R58.1, U21.1
- new net: R52.2, U21.3 (-)
- new net: R55.2, U21.4 (+)
- new net: R50.2, R51.1, U19.5 (ADJ)
- new net: R57.2, U22.3 (-)
- new net: R54.2, U22.4 (+)
- new net +15V_DCCT: R56.2, R57.1
- new net +15V_DCCT_REG: C67.1, C70.1, C71.1, C74.1, R50.1, R54.1, R56.1, U19.4 (OUT), U22.5 (V+)
- new net -15V_DCCT: R53.1, R55.1
- new net -15V_DCCT_REG: C66.1, C68.1, C69.1, C72.1, R52.1, R53.2, U20.4 (SENSE), U20.5 (OUT), U21.2 (V-)

Commit message: Finished layout
Parts:
- added F1, F2: Polyfuse, myparts:FUSE_SMDC300F&slash_24-2_LTF, symbol Device:Polyfuse
- added TP10, TP11: ${SHORT_NET_NAME(1)}, TestPoint:TestPoint_THTPad_D2.0mm_Drill1.0mm, symbol Connector:TestPoint
- C60, C61: footprint CAP_EEFK_D8_PAN -> myparts:CAP_EEFK_D8_PAN; Cost (none) -> 0.44; MFG (none) -> Panasonic; MFG_PN (none) -> EEE-FTH101XAP
- C62, C63, C68, C70: Cost (none) -> .04; MFG (none) -> Samsung; MFG_PN (none) -> CL10A106MA8NRNC
- C64, C65, C69, C71, C72, C73, C74: Cost (none) -> .01; MFG (none) -> Taiyo Yuden; MFG_PN (none) -> TMK105BJ104KV-F
- C66, C67: footprint CAPMP7.6X4.3_4.3N_KEM -> myparts:CAPMP7.6X4.3_4.3N_KEM; Cost (none) -> 3.56; MFG (none) -> Kemet; MFG_PN (none) -> T521X107M025ATE060
- R50: value 11.4K -> 11.5K; Cost (none) -> 0.01; MFG (none) -> Panasonic; MFG_PN (none) -> ERJ-2RKF1152X
- R51: Cost (none) -> 0.01; MFG (none) -> Panasonic; MFG_PN (none) -> ERJ-2RKF1001X
- R52, R54, R55, R57: Cost (none) -> 0.01; MFG (none) -> Panasonic; MFG_PN (none) -> ERJ-2RKF1000X
- R53, R56: value KRL6432E-M-R010-F-T1 -> 0.01; Cost (none) -> 0.71; MFG (none) -> Susumu; MFG_PN (none) -> KRL6432E-M-R010-F-T1
- R58, R59: Cost (none) -> 0.01; MFG (none) -> Panasonic; MFG_PN (none) -> ERJ-2RKF4991X
- U19: Cost (none) -> 5.57; MFG (none) -> Analog Devices; MFG_PN (none) -> LT1963AEQ#TRPBF
- U20: value LT3015xQ-15 -> LT3015EQ-15; Cost (none) -> 6.46; MFG (none) -> Analog Devices; MFG_PN (none) -> LT3015EQ-15#PBF
- U21, U22: value LT6105 -> LT6106; Cost (none) -> 2.01; MFG (none) -> Analog Devices; MFG_PN (none) -> LT6106CS5#TRMPBF
Connections:
- net +15V_DCCT: now also F1.2, TP10.1; no longer R56.2, R57.1
- net -15V_DCCT: now also F2.2, TP11.1; no longer R53.1, R55.1
- net -15V_DCCT_REG: now also C66.2; no longer C66.1
- net -18V: now also C61.2; no longer C61.1
- net GND: now also C61.1, C66.1; no longer C61.2, C66.2
- net +5V renamed +5.0V
- new net +15V_DCCT_uf: F1.1, R56.2, R57.1
- new net -15V_DCCT_uf: F2.1, R53.1, R55.1
Other:
- moved on the sheet: C61, C66
